File: StagX-MaxEdit/StagX.kicad_sch (KiCad schematic)
At the start: 2 parts

Commit message: Updated maxedit after git fun
Other:
- sheet LOOM - Rear Box renamed LOOM - REAR BOX
- removed sheet DEVICE - UMBILICAL
- added sheet LOOM - SIDE PANEL (loom-side-panel.kicad_sch)
- sheet LOOM - FRONT ports: added ROLL HOOP SHUTDOWN, ROLL HOOP TSAL; removed ROLL HOOP
- sheet LOOM - ROLL HOOP ports: added SHUTDOWN, TSAL; removed ROLL HOOP
Changed lines of the file:
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@@
+    (stroke (width 0) (type default))
+  )
+  (bus (pts (xy 323.85 63.5) (xy 331.47 63.5))
     (stroke (width 0) (type default))
   )
@@
     (stroke (width 0) (type default))
   )
-  (bus (pts (xy 227.33 165.1) (xy 233.68 165.1))
+  (bus (pts (xy 227.33 191.77) (xy 233.68 191.77))
     (stroke (width 0) (type default))
   )
@@
     (stroke (width 0) (type default))
   )
-  (bus (pts (xy 227.33 209.55) (xy 227.33 165.1))
+  (bus (pts (xy 227.33 209.55) (xy 227.33 191.77))
     (stroke (width 0) (type default))
   )
@@
     (effects (font (size 1.27 1.27)) (justify left bottom))
   )
-  (text "Check complete shutdown loop" (at 241.3 246.38 0)
+  (text "Check complete shutdown loop" (at 236.22 254 0)
     (effects (font (size 2 2) (thickness 0.4) bold (color 255 0 0 1)) (justify left bottom))
   )
@@
     )
   )
-  (sheet (at 308.61 217.17) (size 19.05 8.89) (fields_autoplaced)
+  (sheet (at 237.49 267.97) (size 19.05 8.89) (fields_autoplaced)
     (stroke (width 0.1524) (type solid) (color 132 0 132 1))
     (fill (color 132 0 132 0.2000))
-    (property "Sheetname" "ACRONYMS" (at 308.61 216.4584 0)
-      (effects (font (size 1.27 1.27)) (justify left bottom))
-    )
-    (property "Sheetfile" "acronyms.kicad_sch" (at 308.61 226.6446 0)
+    (property "Sheetname" "ACRONYMS" (at 237.49 267.2584 0)
+      (effects (font (size 1.27 1.27)) (justify left bottom))
+    )
+    (property "Sheetfile" "acronyms.kicad_sch" (at 237.49 277.4446 0)
       (effects (font (size 1.27 1.27)) (justify left top) hide)
     )
@@
     )
   )
-  (sheet (at 100.33 78.74) (size 53.34 105.41) (fields_autoplaced)
+  (sheet (at 129.54 78.74) (size 24.13 105.41) (fields_autoplaced)
     (stroke (width 0.1524) (type solid))
     (fill (color 0 0 0 0.0000))
-    (property "Sheetname" "LOOM - REAR" (at 100.33 78.0284 0)
-      (effects (font (size 1.27 1.27)) (justify left bottom))
-    )
-    (property "Sheetfile" "loom-rear.kicad_sch" (at 100.33 184.7346 0)
+    (property "Sheetname" "LOOM - REAR" (at 129.54 78.0284 0)
+      (effects (font (size 1.27 1.27)) (justify left bottom))
+    )
+    (property "Sheetfile" "loom-rear.kicad_sch" (at 129.54 184.7346 0)
       (effects (font (size 1.27 1.27)) (justify left top) hide)
     )
@@
     )
   )
-  (sheet (at 331.47 161.29) (size 45.72 33.02) (fields_autoplaced)
+  (sheet (at 331.47 161.29) (size 45.72 19.05) (fields_autoplaced)
     (stroke (width 0.1524) (type solid))
     (fill (color 0 0 0 0.0000))
@@
       (effects (font (size 1.27 1.27)) (justify left bottom))
     )
-    (property "Sheetfile" "loom-dash-box.kicad_sch" (at 331.47 194.8946 0)
+    (property "Sheetfile" "loom-dash-box.kicad_sch" (at 331.47 180.9246 0)
       (effects (font (size 1.27 1.27)) (justify left top) hide)
     )
@@
     )
   )
-  (sheet (at 335.28 198.12) (size 26.67 7.62) (fields_autoplaced)
-    (stroke (width 0.1524) (type solid) (color 0 132 132 1))
-    (fill (color 0 132 132 0.2000))
-    (property "Sheetname" "DEVICE - UMBILICAL" (at 335.28 197.4084 0)
-      (effects (font (size 1.27 1.27)) (justify left bottom))
-    )
-    (property "Sheetfile" "Device-Umbilical.kicad_sch" (at 335.28 206.3246 0)
-      (effects (font (size 1.27 1.27)) (justify left top) hide)
-    )
-    (instances
-      (project "StagX"
-        (path "/03011643-0690-4b85-ab78-d6a62dae52b1" (page "28"))
-      )
-    )
-  )
   (sheet (at 364.49 67.31) (size 26.67 7.62) (fields_autoplaced)
     (stroke (width 0.1524) (type solid) (color 0 132 132 1))
@@
     )
   )
-  (sheet (at 67.31 111.76) (size 27.94 10.16) (fields_autoplaced)
-    (stroke (width 0.1524) (type solid) (color 0 132 132 1))
-    (fill (color 0 132 132 0.2000))
-    (property "Sheetname" "DEVICE - MOTOR" (at 67.31 111.0484 0)
-      (effects (font (size 1.27 1.27)) (justify left bottom))
-    )
-    (property "Sheetfile" "device-motor.kicad_sch" (at 67.31 122.5046 0)
-      (effects (font (size 1.27 1.27)) (justify left top) hide)
-    )
-    (pin "PHASE.V" bidirectional (at 67.31 116.84 180)
-      (effects (font (size 1.27 1.27)) (justify left))
-    )
-    (pin "PHASE.U" bidirectional (at 67.31 114.3 180)
-      (effects (font (size 1.27 1.27)) (justify left))
-    )
-    (pin "PHASE.W" bidirectional (at 67.31 119.38 180)
-      (effects (font (size 1.27 1.27)) (justify left))
-    )
-    (pin "RESOLVER" bidirectional (at 95.25 114.3 0)
-      (effects (font (size 1.27 1.27)) (justify right))
-    )
-    (pin "TEMP" bidirectional (at 95.25 119.38 0)
+  (sheet (at 72.39 198.12) (size 64.77 22.86) (fields_autoplaced)
+    (stroke (width 0.1524) (type solid))
+    (fill (color 0 0 0 0.0000))
+    (property "Sheetname" "LOOM - SIDE PANEL" (at 72.39 197.4084 0)
+      (effects (font (size 1.27 1.27)) (justify left bottom))
+    )
+    (property "Sheetfile" "loom-side-panel.kicad_sch" (at 72.39 221.5646 0)
+      (effects (font (size 1.27 1.27)) (justify left top) hide)
+    )
+    (instances
+      (project "StagX"
+        (path "/03011643-0690-4b85-ab78-d6a62dae52b1" (page "29"))
+      )
+    )
+  )
+  (sheet (at 62.23 115.57) (size 27.94 10.16) (fields_autoplaced)
+    (stroke (width 0.1524) (type solid) (color 0 132 132 1))
+    (fill (color 0 132 132 0.2000))
+    (property "Sheetname" "DEVICE - MOTOR" (at 62.23 114.8584 0)
+      (effects (font (size 1.27 1.27)) (justify left bottom))
+    )
+    (property "Sheetfile" "device-motor.kicad_sch" (at 62.23 126.3146 0)
+      (effects (font (size 1.27 1.27)) (justify left top) hide)
+    )
+    (pin "PHASE.V" bidirectional (at 62.23 120.65 180)
+      (effects (font (size 1.27 1.27)) (justify left))
+    )
+    (pin "PHASE.U" bidirectional (at 62.23 118.11 180)
+      (effects (font (size 1.27 1.27)) (justify left))
+    )
+    (pin "PHASE.W" bidirectional (at 62.23 123.19 180)
+      (effects (font (size 1.27 1.27)) (justify left))
+    )
+    (pin "RESOLVER" bidirectional (at 90.17 118.11 0)
+      (effects (font (size 1.27 1.27)) (justify right))
+    )
+    (pin "TEMP" bidirectional (at 90.17 123.19 0)
       (effects (font (size 1.27 1.27)) (justify right))
     )
@@
     )
   )
-  (sheet (at 349.25 215.9) (size 50.8 22.86) (fields_autoplaced)
+  (sheet (at 341.63 199.39) (size 50.8 22.86) (fields_autoplaced)
     (stroke (width 0.1524) (type solid) (color 204 102 0 1))
     (fill (color 204 102 0 0.2000))
-    (property "Sheetname" "LOOM - CHARGING CART" (at 349.25 215.1884 0)
-      (effects (font (size 1.27 1.27)) (justify left bottom))
-    )
-    (property "Sheetfile" "loom-charging-cart.kicad_sch" (at 349.25 239.3446 0)
+    (property "Sheetname" "LOOM - CHARGING CART" (at 341.63 198.6784 0)
+      (effects (font (size 1.27 1.27)) (justify left bottom))
+    )
+    (property "Sheetfile" "loom-charging-cart.kicad_sch" (at 341.63 222.8346 0)
       (effects (font (size 1.27 1.27)) (justify left top) hide)
     )
@@
     )
   )
-  (sheet (at 308.61 232.41) (size 20.32 11.43) (fields_autoplaced)
+  (sheet (at 269.24 266.7) (size 20.32 11.43) (fields_autoplaced)
     (stroke (width 0.1524) (type solid) (color 132 0 132 1))
     (fill (color 132 0 132 0.2000))
-    (property "Sheetname" "PINOUTS" (at 308.61 231.6984 0)
-      (effects (font (size 1.27 1.27)) (justify left bottom))
-    )
-    (property "Sheetfile" "pinouts.kicad_sch" (at 308.61 244.4246 0)
+    (property "Sheetname" "PINOUTS" (at 269.24 265.9884 0)
+      (effects (font (size 1.27 1.27)) (justify left bottom))
+    )
+    (property "Sheetfile" "pinouts.kicad_sch" (at 269.24 278.7146 0)
       (effects (font (size 1.27 1.27)) (justify left top) hide)
     )
@@
     )
   )
-  (sheet (at 66.04 161.29) (size 27.94 22.86) (fields_autoplaced)
+  (sheet (at 97.79 105.41) (size 27.94 77.47) (fields_autoplaced)
     (stroke (width 0.1524) (type solid))
     (fill (color 0 0 0 0.0000))
-    (property "Sheetname" "LOOM - Rear Box" (at 66.04 160.5784 0)
-      (effects (font (size 1.27 1.27)) (justify left bottom))
-    )
-    (property "Sheetfile" "loom-rear-box.kicad_sch" (at 66.04 184.7346 0)
+    (property "Sheetname" "LOOM - REAR BOX" (at 97.79 104.6984 0)
+      (effects (font (size 1.27 1.27)) (justify left bottom))
+    )
+    (property "Sheetfile" "loom-rear-box.kicad_sch" (at 97.79 183.4646 0)
       (effects (font (size 1.27 1.27)) (justify left top) hide)
     )
@@
       (effects (font (size 1.27 1.27)) (justify right))
     )
-    (pin "ROLL HOOP" bidirectional (at 331.47 58.42 180)
+    (pin "TSAL" bidirectional (at 331.47 58.42 180)
+      (effects (font (size 1.27 1.27)) (justify left))
+    )
+    (pin "SHUTDOWN" bidirectional (at 331.47 63.5 180)
       (effects (font (size 1.27 1.27)) (justify left))
     )
@@
       (effects (font (size 1.27 1.27)) (justify left))
     )
-    (pin "COCKPIT E-STOP" bidirectional (at 233.68 165.1 180)
-      (effects (font (size 1.27 1.27)) (justify left))
-    )
-    (pin "ROLL HOOP" bidirectional (at 323.85 58.42 0)
-      (effects (font (size 1.27 1.27)) (justify right))
+    (pin "COCKPIT E-STOP" bidirectional (at 233.68 191.77 180)
+      (effects (font (size 1.27 1.27)) (justify left))
     )
     (pin "UMBILICAL" bidirectional (at 323.85 191.77 0)
       (effects (font (size 1.27 1.27)) (justify right))
     )
+    (pin "ROLL HOOP SHUTDOWN" bidirectional (at 323.85 63.5 0)
+      (effects (font (size 1.27 1.27)) (justify right))
+    )
+    (pin "ROLL HOOP TSAL" bidirectional (at 323.85 58.42 0)
+      (effects (font (size 1.27 1.27)) (justify right))
+    )

Commit message: Added initial version for loom routing
Parts:
- removed D?: BRAKE LIGHT, symbol Device:LED_Series
- removed FAN?: REAR RADIATOR FAN, symbol Motor:Fan
- added BATT?: ~, symbol Device:Battery
- added F?: 10A, symbol Device:Fuse
Connections:
- new net: BATT?.1 (+), F?.1
- new net DEVICE - GROUND BOX/BATT GND: BATT?.2 (-)
- new net LOOM - SIDE PANEL/LVS.MAIN.EXC: F?.2
Other:
- added sheet DEVICE - BRAKE LIGHT (device-brake-light.kicad_sch)
- added sheet DEVICE - BSPD (device-bspd.kicad_sch)
- added sheet DEVICE - CURRENT SENSOR (device-current-sensor.kicad_sch)
- added sheet DEVICE - GROUND BOX (device-ground-box.kicad_sch)
- added sheet DEVICE - RADIATOR FAN (device-radiator-fan.kicad_sch)
- sheet DEVICE - SAGL: file device-bspd.kicad_sch -> device-sagl.kicad_sch
- sheet LOOM - ACCUMULATOR ports: added CAR I/O, CHARGER I/O, DC.+, DC.-; removed none
- sheet LOOM - FRONT ports: added DASH LEDS; removed none
- sheet LOOM - PEDAL BOX ports: added BSPD; removed none
- sheet LOOM - REAR ports: added ACCUMULATOR, BRAKE LIGHT, BSPD CT, FAN, FIREWALL, GND BOX, INVERTER CASING, INVERTER J1, INVERTER J2, MOTOR RESOLVER, MOTOR TEMP, PDM A, PDM B, PUMP 1, PUMP 2, REAR BOX, SIDEPANEL; removed none
- sheet LOOM - REAR BOX ports: added HV1, HV2, HV3, HV4, REAR BOX I/O, TSMP.HV+, TSMP.HV-; removed none
- sheet LOOM - SIDE PANEL ports: added LVS.MAIN.EXC, LVS.MAIN.SWITCHED.EXC, SIDE PANEL, TSMP HV+, TSMP HV-; removed none
- note added: "FINISH HV WIRES"
- note added: "NOTES: 1. GRID SIZE = 1.27MM 2. THICK ORANGE CABLES INDICATE 35MM2 CABLING ON CAR"
- note removed: "NOTES: 1. EXAMPLE NOTE"
