File: StagX-MaxEdit/loom-accumulator.kicad_sch (KiCad schematic)
At the start: 20 parts

Commit message: Updated maxedit after git fun
Parts:
- added SP? (x6): GND, symbol Connector:TestPoint_Small
- renumbered CONN to CONN?, Conn1 to Conn?, SP1 to SP?, SP2 to SP?, SP3 to SP?
Connections:
- net BMS.EXC is gone; now on net BMS.Charge.EXC: CONN?.2 (Pin_2)
- net SHUT.OUT is gone; now on net +AIR.GND: Conn?.1
- net BMS.Charge.EXC: now also SP?.1
- net CAN.S.HIGH: now also SP?.1
- net CAN.S.LOW: now also SP?.1
- net IMD.EXC: now also SP?.1
- net ISOLATOR.EXC: now also SP?.1
- net SHUT.IN: now also SP?.1
- net TSAC.HVS.BATT.EXC renamed TSAC.HVS.EXC
- net TSAC.HVS.BATT.GND renamed TSAC.HVS.GND
Other:
- note added: "Check this doesn't have wires already that we need to solder to instead"
- note added: "Ring terminals onto splices"
- note removed: "Check this doesn't have wires already"
- moved on the sheet: Conn?

Commit message: Added initial version for loom routing
Parts:
- removed Conn? (x3): Deutsch_DTM_4P_Pin, symbol Connectors_SUFST:Deutsch_DTM_4P_Pin
- added Conn1, Conn2, Conn3: Deutsch_DTM_4S_Pin, symbol Connectors_SUFST:Deutsch_DTM_4S_Pin
- added Conn?: AMPHENOL-21P-Pannel, symbol Connectors_SUFST:AMPHENOL-21P-Pannel
- added Conn?: AMPHENOL-47P-Pannel, symbol Connectors_SUFST:AMPHENOL-47P-Pannel
- added F?: 100A, symbol Device:Fuse
Connections:
- net +AIR.AUX.EXC: now also Conn1.2, Conn?.28
- net +AIR.AUX.GND: now also Conn1.1, Conn?.29
- net +AIR.EXC: now also Conn1.4
- net +AIR.GND: now also Conn1.3, Conn2.2, Conn?.1, Conn?.1, Conn?.2, Conn?.2
- net +AIR.INTENDED.ON: now also Conn?.21
- net -AIR.AUX.EXC: now also Conn2.3, Conn?.26
- net -AIR.AUX.GND: now also Conn2.4, Conn?.27
- net -AIR.EXC: now also Conn2.1, Conn?.14
- net -AIR.INTENDED.ON: now also Conn?.22
- net BMS.CHARGER.SAFETY: now also Conn?.9
- net BMS.CUR_SEN.GND: now also Conn?.3; no longer Conn?.2
- net BMS.CUR_SEN.HIGH: now also Conn?.2; no longer Conn?.3
- net BMS.Charge.EXC: now also Conn?.4, Conn?.4
- net BMS.FAULT: now also Conn?.31
- net CAN.S.HIGH: now also Conn?.11, Conn?.6, Conn?.9
- net CAN.S.LOW: now also Conn?.10, Conn?.12, Conn?.7
- net CHASSIS.GND: now also Conn?.15
- net IMD.EXC: now also Conn?.5, Conn?.5
- net IMD.OK: now also Conn?.16
- net INV.CLOSE.+AIR: now also Conn?.19
- net INV.CLOSE.PCHG: now also Conn?.20
- net ISOLATOR.EXC: now also Conn?.3, Conn?.3
- net PCHG.AUX.EXC: now also Conn3.3, Conn?.24
- net PCHG.AUX.GND: now also Conn3.4, Conn?.25
- net PCHG.EXC: now also Conn3.1
- net PCHG.GND: now also Conn3.2
- net PCHG.INTENDED.ON: now also Conn?.23
- net SHUT.IN: now also Conn?.13, Conn?.8
- net TS.ON: now also Conn?.18
- net TS.READY: now also Conn?.17
- net TSAC.HVS.EXC: now also Conn?.6
- net TSAC.HVS.GND: now also Conn?.7
- net ~{BMS.CHARGER.INTERLOCKED}: now also Conn?.10
- net ~{BMS.DISCHARGE.ENABLE}: now also Conn?.30
- net ~{TS.DETECTED}: now also Conn?.8
- no-connect marks 51 -> 78
Other:
- note added: "ALL SPLICES ARE RING TERMINALS ON AIRS"
- note added: "Add devices"
- note added: "CHECK FUSE VALUE"
- note added: "Change how HV splices work to be over the isolation line and physically connecting o the airs and precharge etc"
- note added: "Expecting new precharge to go here"
- note added: "HV CONNECTIONS"
- note added: "HV SENSE"
- note added: "NEEDS HV CONNECTOR INTERLOCK ADDED"
- note added: "PRECHARGE"
- note added: "RING TERMINAL ON AIR"
- note removed: "HV_Sense"
- note removed: "Is this active low?"
- note removed: "Ring terminals onto splices"
- note removed: "SPLICE on ring terminal"
- title: (none) -> LOOM - ACCUMULATOR
- moved on the sheet: CONN?, Conn?, SP?
