File: StagX-MaxEdit/loom-charging-cart.kicad_sch (KiCad schematic)
At the start: 0 parts

Commit message: Added initial version for loom routing
Other:
- note added: "Charger Umbilical Separate "shore" power? Charging e-stop loop switches and LED indicators"
- title: (none) -> LOOM - CHARGING CART
Changed lines of the file:
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@@
 (kicad_sch (version 20230121) (generator eeschema)
   (paper "A4")
+  (title_block
+    (title "LOOM - CHARGING CART")
+  )
+  (text "Charger\nUmbilical\nSeparate \"shore\" power?\nCharging e-stop loop\nswitches and LED indicators"
+    (at 134.62 78.74 0)
+    (effects (font (size 1.27 1.27)) (justify left bottom))
+  )
 )
