File: StagX-MaxEdit/loom-dash-box.kicad_sch (KiCad schematic)
At the start: 17 parts

Commit message: Added initial version for loom routing
Parts:
- renumbered Conn20 to Conn?, SP6 to SP?, SP5 to SP?, SP4 to SP?, SP to SP?
Connections:
- net L120.SENSOR.5V.EXC: now reaches Conn?.27
- net L120.SENSOR.5V.EXC: now also Conn?.8
- net L120.SENSOR.GND: now reaches Conn?.28
- net L120.SENSOR.GND: now also Conn?.9
- net L120.ANALOGUE.VOLT.1: now reaches Conn?.29
- net L120.ANALOGUE.VOLT.1: now also Conn?.4
- net L120.ANALOGUE.VOLT.2: now reaches Conn?.30
- net L120.ANALOGUE.VOLT.2: now also Conn?.5
- net L120.ANALOGUE.VOLT.3: now reaches Conn?.31
- net L120.ANALOGUE.VOLT.3: now also Conn?.6
- net L120.ANALOGUE.VOLT.4: now reaches Conn?.32
- net L120.ANALOGUE.VOLT.4: now also Conn?.7
- net L120.ANALOGUE.VOLT.5: now reaches Conn?.33
- net L120.ANALOGUE.VOLT.5: now also Conn?.12
- net L120.ANALOGUE.VOLT.6: now reaches Conn?.34
- net L120.ANALOGUE.VOLT.6: now also Conn?.13
- net L120.DIGITAL.1: now reaches Conn?.35
- net L120.DIGITAL.1: now also Conn?.14
- net L120.DIGITAL.2: now reaches Conn?.36
- net L120.DIGITAL.2: now also Conn?.15
- net L120.ANALOGUE.TEMP.1: now reaches Conn?.37
- net L120.ANALOGUE.TEMP.1: now also Conn?.16
- net L120.ANALOGUE.TEMP.2: now reaches Conn?.38
- net L120.ANALOGUE.TEMP.2: now also Conn?.17
- net L120.SPEED.1: now reaches Conn?.39
- net L120.SPEED.1: now also Conn?.21
- net L120.SPEED.2: now reaches Conn?.40
- net L120.SPEED.2: now also Conn?.22
- net L120.SPEED.3: now reaches Conn?.41
- net L120.SPEED.3: now also Conn?.23
- no-connect marks 37 -> 30
Other:
- note added: "25mA MAXIMUM RECOMMENDED TO USE EXTERNAL POWER"
- note added: "sensors that may need to connect to this: - wheel speed sensors - damper pots"
- note removed: "sensors that may need to connect to this: - wheel speed sensors - dampner pots"
- title: (none) -> LOOM - DASH BOX
- moved on the sheet: Conn?, SP?
