File: StagX-MaxEdit/loom-rear-box.kicad_sch (KiCad schematic)
At the start: 0 parts

Commit message: Updated maxedit after git fun
Parts:
- added B?: +VE Busbar, symbol Connectors_SUFST:Bus_Bar
- added B?: HVD, symbol Connectors_SUFST:Bus_Bar
- added BATT?: TSAL BATTERY, symbol Device:Battery
- added CONN?: HVD_INTERLOCK, symbol Connector:Conn_01x02_Socket
- added Conn? (x8): Molex_2x1P_Horizontal_THT, symbol Connectors_SUFST:Molex_2x1P_Horizontal_THT
- added Conn?: ~, symbol Connectors_SUFST:Molex_2x2P_Horizontal
- added Conn? (x6): Molex_2x2P_Horizontal, symbol Connectors_SUFST:Molex_2x2P_Horizontal
- added Conn? (x2): Molex_6x1P_Horizontal_THT, symbol Connectors_SUFST:Molex_6x1P_Horizontal_THT
- added R? (x2): 15k, symbol Device:R_Small
Connections:
- new net: B?.4 (S2), R?.2 (x2)
- new net +AIR.AUX.EXC: Conn?.2
- new net +AIR.AUX.GND: Conn?.5
- new net +AIR.INTENDED.ON: Conn?.2
- new net -AIR.AUX.EXC: Conn?.1
- new net -AIR.AUX.GND: Conn?.4
- new net -AIR.INTENDED.ON: Conn?.1
- new net BATT+: BATT?.1 (+), Conn?.1
- new net BATT-: BATT?.2 (-), Conn?.2
- new net BMS.FAULT: Conn?.2
- new net BMS.FAULT.LATCHING: Conn?.2
- new net COCKPIT.TS.LED.GND: Conn?.4
- new net Discharge.HV+: B?.5 (S3), Conn?.1
- new net Discharge.HV-: B?.5 (S3), Conn?.2
- new net HVS.HV+: B?.3 (S1), Conn?.1
- new net HVS.HV-: B?.3 (S1), Conn?.2
- new net IMD.FAULT.LATCHING: Conn?.1
- new net IMD.OK: Conn?.3
- new net LATCHING.EXC: Conn?.1
- new net LATCHING.GND: Conn?.2
- new net LATCHING.RESET+: Conn?.1
- new net LATCHING.RESET-: Conn?.2
- new net PCHG.AUX.EXC: Conn?.3
- new net PCHG.AUX.GND: Conn?.6
- new net PCHG.INTENDED.ON: Conn?.3
- new net REB.HVS.EXC: Conn?.3, Conn?.3
- new net REB.HVS.GND: Conn?.4, Conn?.4
- new net SHUT.DISCHARGE: Conn?.1
- new net SHUT.GND: Conn?.2
- new net SHUT.HVD.INTERLOCK: CONN?.1 (Pin_1)
- new net SHUT.LATCHING: CONN?.2 (Pin_2), Conn?.3
- new net SHUT.TSMS: Conn?.4
- new net TS.DETECTED: Conn?.1, Conn?.1
- new net TSAC.HVS.EXC: Conn?.3
- new net TSAC.HVS.GND: Conn?.4
- new net TSAL.EXC: Conn?.3
- new net TSAL.GND: Conn?.4
- new net TSAL.GREEN.LED.GND: Conn?.2
- new net TSAL.LED.EXC: Conn?.1
- new net TSAL.RED.LED.GND: Conn?.3
- new net TSAL.RESET+: Conn?.2
- new net TSAL.RESET-: Conn?.1
- new net TSMP.HV+: R?.1
- new net TSMP.HV-: R?.1
- new net ~{BMS.DISCHARGE.ENABLE}: Conn?.1
- new net ~{TS.DETECTED}: Conn?.2
- no-connect marks 0 -> 11
Other:
- note added: "Change to socket molex"
- note added: "DISCHARGE"
- note added: "HV SENSE"
- note added: "HVD"
- note added: "IMD"
- note added: "New HVD symbol?"
- note added: "Re-do busbar symbol to be on grid Connect HV sheet pins"
- note added: "TSAL"
- note added: "TSMPs"

Commit message: Added initial version for loom routing
Parts:
- added Conn?: AMPHENOL-47P-Pannel, symbol Connectors_SUFST:AMPHENOL-47P-Pannel
- added Conn?: Current Sensor, symbol Connectors_SUFST:Current Sensor Connector
Connections:
- net +AIR.AUX.EXC: now also Conn?.4
- net +AIR.AUX.GND: now also Conn?.7
- net +AIR.INTENDED.ON: now also Conn?.10
- net -AIR.AUX.EXC: now also Conn?.3
- net -AIR.AUX.GND: now also Conn?.6
- net -AIR.INTENDED.ON: now also Conn?.9
- net BMS.FAULT: now also Conn?.26
- net BMS.FAULT.LATCHING: now also Conn?.22
- net COCKPIT.TS.LED.GND: now also Conn?.17
- net IMD.FAULT.LATCHING: now also Conn?.21
- net IMD.OK: now also Conn?.27
- net LATCHING.EXC: now also Conn?.28
- net LATCHING.GND: now also Conn?.29
- net LATCHING.RESET+: now also Conn?.23
- net LATCHING.RESET-: now also Conn?.24
- net PCHG.AUX.EXC: now also Conn?.5
- net PCHG.AUX.GND: now also Conn?.8
- net PCHG.INTENDED.ON: now also Conn?.11
- net SHUT.DISCHARGE: now also Conn?.35
- net SHUT.GND: now also Conn?.36
- net SHUT.HVD.INTERLOCK: now also Conn?.34
- net SHUT.TSMS: now also Conn?.33
- net TSAC.HVS.EXC: now also Conn?.19
- net TSAC.HVS.GND: now also Conn?.20
- net TSAL.EXC: now also Conn?.1
- net TSAL.GND: now also Conn?.2
- net TSAL.GREEN.LED.GND: now also Conn?.15
- net TSAL.LED.EXC: now also Conn?.14
- net TSAL.RED.LED.GND: now also Conn?.16
- net TSAL.RESET+: now also Conn?.13
- net TSAL.RESET-: now also Conn?.12
- net ~{BMS.DISCHARGE.ENABLE}: now also Conn?.25
- net ~{TS.DETECTED}: now also Conn?.18
- net Discharge.HV+ renamed DISCHARGE.HV+
- net Discharge.HV- renamed DISCHARGE.HV-
- new net BSPD.CUR_SEN.EXC: Conn?.1, Conn?.30
- new net BSPD.CUR_SEN.GND: Conn?.3, Conn?.32
- new net BSPD.CUR_SEN.SIG: Conn?.31, Conn?.4
- no-connect marks 11 -> 23
Other:
- note added: "Ampllifier route power "around" this"
- note added: "CURRENT SENSOR"
- note added: "LATCHING"
- note added: "LOW RANGE USED"
- note added: "SITS AROUND HVD BUSBARS"
- note removed: "IMD"
- title: (none) -> LOOM - REAR BOX
- moved on the sheet: B?, CONN?, Conn?, R?
