File: StagX/loom-rear.kicad_sch (KiCad schematic)
At the start: 16 parts

Commit message: Completed shutdown loop
Parts:
- added J?: RING TERMINAL ON MAIN ROLL HOOP, symbol Connector_Generic:Conn_01x01
Connections:
- net SHUT.TRC is gone; now on net SHUT.TSAC.INTERLOCK: Conn?.13
- net CHASSIS.GND: now also J?.1 (Pin_1)
- net RS-232.GND: now also Conn?.22
- net GND: no longer names the net of Conn?.19
- no-connect marks 51 -> 48
Other:
- note added: "SPLICE AT RESISTOR"
- note removed: "RS232 GND"
- note removed: "SHUTDOWN LOOP IS MISSING"
Changed lines of the file:
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@@
   (no_connect (at 43.18 124.46))
   (no_connect (at 539.75 121.92))
-  (no_connect (at 513.08 212.09))
   (no_connect (at 539.75 129.54))
   (no_connect (at 513.08 242.57))
@@
   (no_connect (at 539.75 119.38))
   (no_connect (at 43.18 144.78))
-  (no_connect (at 513.08 214.63))
   (no_connect (at 43.18 129.54))
   (no_connect (at 539.75 137.16))
@@
   (no_connect (at 539.75 142.24))
   (no_connect (at 539.75 111.76))
-  (no_connect (at 513.08 217.17))
   (no_connect (at 539.75 139.7))
   (no_connect (at 513.08 234.95))
@@
   (no_connect (at 513.08 219.71))
   (no_connect (at 513.08 227.33))
+  (wire (pts (xy 539.75 66.04) (xy 506.73 66.04))
+    (stroke (width 0) (type default))
+  )
   (wire (pts (xy 68.58 388.62) (xy 193.04 388.62))
     (stroke (width 0) (type default))
@@
     (stroke (width 0) (type default))
   )
+  (wire (pts (xy 455.93 223.52) (xy 158.75 223.52))
+    (stroke (width 0) (type default))
+  )
   (wire (pts (xy 455.93 241.3) (xy 410.21 241.3))
     (stroke (width 0) (type default))
@@
     (stroke (width 0) (type default))
   )
+  (wire (pts (xy 415.29 226.06) (xy 455.93 226.06))
+    (stroke (width 0) (type default))
+  )
   (wire (pts (xy 130.81 161.29) (xy 130.81 186.69))
     (stroke (width 0) (type default))
@@
     (stroke (width 0) (type default))
   )
+  (wire (pts (xy 513.08 217.17) (xy 260.35 217.17))
+    (stroke (width 0) (type default))
+  )
   (wire (pts (xy 68.58 156.21) (xy 146.05 156.21))
     (stroke (width 0) (type default))
   )
+  (wire (pts (xy 135.89 86.36) (xy 135.89 181.61))
+    (stroke (width 0) (type default))
+  )
   (wire (pts (xy 513.08 146.05) (xy 373.38 146.05))
     (stroke (width 0) (type default))
@@
     (stroke (width 0) (type default))
   )
+  (wire (pts (xy 158.75 223.52) (xy 158.75 60.96))
+    (stroke (width 0) (type default))
+  )
   (wire (pts (xy 303.53 55.88) (xy 303.53 280.67))
     (stroke (width 0) (type default))
@@
     (stroke (width 0) (type default))
   )
+  (wire (pts (xy 415.29 209.55) (xy 415.29 226.06))
+    (stroke (width 0) (type default))
+  )
   (wire (pts (xy 455.93 238.76) (xy 412.75 238.76))
     (stroke (width 0) (type default))
@@
     (stroke (width 0) (type default))
   )
+  (wire (pts (xy 161.29 58.42) (xy 161.29 212.09))
+    (stroke (width 0) (type default))
+  )
+  (wire (pts (xy 135.89 181.61) (xy 68.58 181.61))
+    (stroke (width 0) (type default))
+  )
   (wire (pts (xy 151.13 81.28) (xy 151.13 214.63))
     (stroke (width 0) (type default))
@@
     (stroke (width 0) (type dot))
   )
+  (wire (pts (xy 539.75 63.5) (xy 464.82 63.5))
+    (stroke (width 0) (type default))
+  )
   (polyline (pts (xy 459.74 262.89) (xy 486.41 262.89))
     (stroke (width 0) (type dot))
@@
     (stroke (width 0) (type default))
   )
+  (wire (pts (xy 506.73 66.04) (xy 506.73 22.86))
+    (stroke (width 0) (type default))
+  )
   (wire (pts (xy 455.93 369.57) (xy 406.4 369.57))
     (stroke (width 0) (type default))
@@
     (stroke (width 0) (type default))
   )
+  (wire (pts (xy 464.82 214.63) (xy 513.08 214.63))
+    (stroke (width 0) (type default))
+  )
   (wire (pts (xy 455.93 367.03) (xy 408.94 367.03))
     (stroke (width 0) (type default))
@@
     (stroke (width 0) (type default))
   )
+  (wire (pts (xy 506.73 22.86) (xy 535.94 22.86))
+    (stroke (width 0) (type default))
+  )
   (wire (pts (xy 176.53 166.37) (xy 513.08 166.37))
     (stroke (width 0) (type default))
@@
     (stroke (width 0) (type default))
   )
+  (wire (pts (xy 260.35 359.41) (xy 455.93 359.41))
+    (stroke (width 0) (type default))
+  )
   (polyline (pts (xy 459.74 349.25) (xy 486.41 349.25))
     (stroke (width 0) (type dot))
@@
     (stroke (width 0) (type default))
   )
+  (wire (pts (xy 260.35 217.17) (xy 260.35 359.41))
+    (stroke (width 0) (type default))
+  )
   (wire (pts (xy 408.94 321.31) (xy 455.93 321.31))
     (stroke (width 0) (type default))
   )
+  (wire (pts (xy 43.18 58.42) (xy 161.29 58.42))
+    (stroke (width 0) (type default))
+  )
   (wire (pts (xy 513.08 151.13) (xy 358.14 151.13))
     (stroke (width 0) (type default))
@@
     (stroke (width 0) (type default))
   )
+  (wire (pts (xy 539.75 60.96) (xy 417.83 60.96))
+    (stroke (width 0) (type default))
+  )
   (wire (pts (xy 373.38 146.05) (xy 373.38 91.44))
     (stroke (width 0) (type default))
@@
     (stroke (width 0) (type default))
   )
+  (wire (pts (xy 43.18 86.36) (xy 135.89 86.36))
+    (stroke (width 0) (type default))
+  )
   (wire (pts (xy 368.3 140.97) (xy 368.3 96.52))
     (stroke (width 0) (type default))
@@
     (stroke (width 0) (type default))
   )
+  (wire (pts (xy 161.29 212.09) (xy 513.08 212.09))
+    (stroke (width 0) (type default))
+  )
   (wire (pts (xy 257.81 392.43) (xy 257.81 231.14))
     (stroke (width 0) (type default))
@@
     (stroke (width 0) (type default))
   )
+  (wire (pts (xy 513.08 209.55) (xy 415.29 209.55))
+    (stroke (width 0) (type default))
+  )
   (wire (pts (xy 455.93 397.51) (xy 207.01 397.51))
     (stroke (width 0) (type default))
@@
     (stroke (width 0) (type dot))
   )
+  (wire (pts (xy 464.82 63.5) (xy 464.82 214.63))
+    (stroke (width 0) (type default))
+  )
   (polyline (pts (xy 459.74 288.29) (xy 486.41 288.29))
     (stroke (width 0) (type dot))
@@
     (stroke (width 0) (type default))
   )
+  (wire (pts (xy 417.83 228.6) (xy 455.93 228.6))
+    (stroke (width 0) (type default))
+  )
   (wire (pts (xy 68.58 163.83) (xy 163.83 163.83))
     (stroke (width 0) (type default))
@@
     (stroke (width 0) (type default))
   )
+  (wire (pts (xy 158.75 60.96) (xy 43.18 60.96))
+    (stroke (width 0) (type default))
+  )
   (wire (pts (xy 455.93 377.19) (xy 234.95 377.19))
     (stroke (width 0) (type default))
@@
     (stroke (width 0) (type default))
   )
+  (wire (pts (xy 417.83 60.96) (xy 417.83 228.6))
+    (stroke (width 0) (type default))
+  )
   (wire (pts (xy 190.5 375.92) (xy 68.58 375.92))
     (stroke (width 0) (type default))
@@
     (stroke (width 0) (type default))
   )
-  (rectangle (start 127 184.15) (end 135.89 189.23)
-    (stroke (width 0) (type default) (color 255 0 0 1))
-    (fill (type color) (color 255 0 0 0.2))
-  )
   (rectangle (start 46.99 355.6) (end 86.36 405.13)
     (stroke (width 0) (type default))
@@
     (effects (font (size 1.27 1.27)) (justify left bottom))
   )
+  (text "SPLICE AT\nRESISTOR" (at 119.38 186.69 0)
+    (effects (font (size 1.27 1.27)) (justify left bottom))
+  )
   (text "OUT 8.15" (at 478.79 290.83 0)
     (effects (font (size 1.27 1.27)) (justify left bottom))
@@
     (effects (font (size 1.27 1.27)) (justify left bottom))
   )
-  (text "SHUTDOWN LOOP IS MISSING" (at 200.66 217.17 0)
-    (effects (font (size 4 4) (thickness 0.8) bold (color 255 0 0 1)) (justify left bottom))
-  )
   (text "OUT 8.13" (at 478.79 285.75 0)
     (effects (font (size 1.27 1.27)) (justify left bottom))
@@
     (effects (font (size 1.27 1.27)) (justify left bottom))
   )
-  (text "RS232 GND" (at 64.77 85.09 0)
-    (effects (font (size 2 2) (thickness 0.4) bold (color 255 0 0 1)) (justify left bottom))
-  )
   (text "OUT 20.2" (at 481.33 336.55 0)
     (effects (font (size 1.27 1.27)) (justify left bottom))
@@
     (effects (font (size 1.27 1.27)) (justify right bottom))
   )
+  (label "SHUT.TSAC.INTERLOCK" (at 539.75 60.96 180) (fields_autoplaced)
+    (effects (font (size 1.27 1.27)) (justify right bottom))
+  )
   (label "MOTOR.TEMP.EXC" (at 68.58 161.29 0) (fields_autoplaced)
     (effects (font (size 1.27 1.27)) (justify left bottom))
@@
     (effects (font (size 1.27 1.27)) (justify left bottom))
   )
-  (label "SHUT.TRC" (at 539.75 60.96 180) (fields_autoplaced)
-    (effects (font (size 1.27 1.27)) (justify right bottom))
-  )
   (label "BSPD.CUR_SEN.GND" (at 68.58 163.83 0) (fields_autoplaced)
     (effects (font (size 1.27 1.27)) (justify left bottom))
@@
     (effects (font (size 1.27 1.27)) (justify right bottom))
   )
-  (label "GND" (at 68.58 270.51 0) (fields_autoplaced)
-    (effects (font (size 1.27 1.27)) (justify left bottom))
-  )
   (label "TS.ON" (at 43.18 55.88 0) (fields_autoplaced)
     (effects (font (size 1.27 1.27)) (justify left bottom))
@@
     (effects (font (size 1.27 1.27)) (justify left bottom))
   )
+  (label "RS-232.GND" (at 68.58 181.61 0) (fields_autoplaced)
+    (effects (font (size 1.27 1.27)) (justify left bottom))
+  )
   (label "CAN.S.HIGH" (at 455.93 280.67 180) (fields_autoplaced)
     (effects (font (size 1.27 1.27)) (justify right bottom))
@@
   )
   (label "LATCHING.RESET+" (at 455.93 241.3 180) (fields_autoplaced)
+    (effects (font (size 1.27 1.27)) (justify right bottom))
+  )
+  (label "SHUT.GND" (at 455.93 359.41 180) (fields_autoplaced)
     (effects (font (size 1.27 1.27)) (justify right bottom))
   )
@@
         )
       )
+    )
+  )
+  (symbol (lib_id "Connector_Generic:Conn_01x01") (at 541.02 22.86 0) (unit 1)
+    (in_bom yes) (on_board yes) (dnp no) (fields_autoplaced)
+    (property "Reference" "J?" (at 543.56 21.59 0)
+      (effects (font (size 1.27 1.27)) (justify left))
+    )
+    (property "Value" "RING TERMINAL ON MAIN ROLL HOOP" (at 543.56 24.13 0)
+      (effects (font (size 1.27 1.27)) (justify left))
+    )
+    (property "Footprint" "" (at 541.02 22.86 0)
+      (effects (font (size 1.27 1.27)) hide)
+    )
+    (property "Datasheet" "~" (at 541.02 22.86 0)
+      (effects (font (size 1.27 1.27)) hide)
+    )
+    (property "Conn Name" "" (at 541.02 22.86 0)
+      (effects (font (size 1.27 1.27)))
+    )
+    (pin "1")
+    (instances
+      (project "StagX"
+        (path "/03011643-0690-4b85-ab78-d6a62dae52b1/4eb1cfc3-f934-459f-8af2-f057ec5d36cb"
+          (reference "J?") (unit 1)
+        )
+      )

Commit message: Post comp commit
Connections:
- net TSAC.HVS.GND is gone; now on net TSAC.HVS.EXC: Conn?.20, Conn?.7
- net BSPD.CUR_SEN.EXC: now also Conn?.27; no longer Conn?.26
- net BSPD.CUR_SEN.GND: now also Conn?.28; no longer Conn?.15
- net TSAC.HVS.EXC: now also Conn?.29
- no-connect marks 48 -> 45
Other:
- note added: "1, 4, 5, 6, 34"
Changed lines of the file:
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@@
 		(color 0 0 0 0)
 	)
+	(junction
+		(at 386.08 173.99)
+		(diameter 0)
+		(color 0 0 0 0)
+	)
 	(no_connect
 		(at 43.18 127)
@@
 	)
 	(no_connect
-		(at 43.18 96.52)
-	)
-	(no_connect
 		(at 43.18 119.38)
 	)
@@
 	)
 	(no_connect
-		(at 43.18 99.06)
-	)
-	(no_connect
 		(at 43.18 142.24)
 	)
@@
 	)
 	(no_connect
-		(at 43.18 93.98)
-	)
-	(no_connect
 		(at 539.75 144.78)
 	)
@@
 	(wire
 		(pts
-			(xy 168.91 201.93) (xy 168.91 191.77)
+			(xy 163.83 96.52) (xy 163.83 207.01)
 		)
 		(stroke
@@
 	(wire
 		(pts
-			(xy 265.43 35.56) (xy 43.18 35.56)
+			(xy 168.91 93.98) (xy 168.91 201.93)
 		)
 		(stroke
@@
 	(wire
 		(pts
-			(xy 513.08 143.51) (xy 363.22 143.51)
+			(xy 265.43 35.56) (xy 43.18 35.56)
 		)
 		(stroke
@@
 	(wire
 		(pts
-			(xy 68.58 252.73) (xy 104.14 252.73)
+			(xy 513.08 143.51) (xy 363.22 143.51)
 		)
 		(stroke
@@
 	(wire
 		(pts
-			(xy 68.58 309.88) (xy 101.6 309.88)
+			(xy 68.58 252.73) (xy 104.14 252.73)
 		)
 		(stroke
@@
 	(wire
 		(pts
-			(xy 68.58 191.77) (xy 168.91 191.77)
+			(xy 68.58 309.88) (xy 101.6 309.88)
 		)
 		(stroke
@@
 	(wire
 		(pts
-			(xy 163.83 163.83) (xy 163.83 207.01)
-		)
-		(stroke
-			(width 0)
-			(type default)
-		)
-	)
-	(wire
-		(pts
 			(xy 146.05 83.82) (xy 43.18 83.82)
 		)
@@
 	(wire
 		(pts
+			(xy 43.18 99.06) (xy 340.36 99.06)
+		)
+		(stroke
+			(width 0)
+			(type default)
+		)
+	)
+	(wire
+		(pts
 			(xy 68.58 275.59) (xy 327.66 275.59)
 		)
@@
 	(wire
 		(pts
+			(xy 340.36 99.06) (xy 340.36 173.99)
+		)
+		(stroke
+			(width 0)
+			(type default)
+		)
+	)
+	(wire
+		(pts
 			(xy 408.94 321.31) (xy 455.93 321.31)
 		)
@@
 	(wire
 		(pts
+			(xy 43.18 96.52) (xy 163.83 96.52)
+		)
+		(stroke
+			(width 0)
+			(type default)
+		)
+	)
+	(wire
+		(pts
 			(xy 513.08 151.13) (xy 358.14 151.13)
 		)
@@
 	(wire
 		(pts
+			(xy 340.36 173.99) (xy 386.08 173.99)
+		)
+		(stroke
+			(width 0)
+			(type default)
+		)
+	)
+	(wire
+		(pts
 			(xy 43.18 91.44) (xy 237.49 91.44)
 		)
@@
 		)
 	)
-	(wire
-		(pts
-			(xy 68.58 163.83) (xy 163.83 163.83)
-		)
-		(stroke
-			(width 0)
-			(type default)
-		)
-	)
 	(polyline
 		(pts
@@
 	(wire
 		(pts
+			(xy 43.18 93.98) (xy 168.91 93.98)
+		)
+		(stroke
+			(width 0)
+			(type default)
+		)
+	)
+	(wire
+		(pts
 			(xy 201.93 63.5) (xy 231.14 63.5)
 		)
@@
 		)
 	)
+	(text "1, 4, 5, 6, 34"
+		(exclude_from_sim no)
+		(at 568.96 46.99 0)
+		(effects
+			(font
+				(size 2 2)
+				(thickness 0.4)
+				(bold yes)
+			)
+		)
+	)
 	(text "OUT 8.13"
 		(exclude_from_sim no)
@@
 	)
 	(label "BSPD.CUR_SEN.EXC"
-		(at 68.58 191.77 0)
+		(at 43.18 93.98 0)
 		(fields_autoplaced yes)
 		(effects
@@
 	)
 	(label "BSPD.CUR_SEN.GND"
-		(at 68.58 163.83 0)
+		(at 43.18 96.52 0)
 		(fields_autoplaced yes)
 		(effects
@@
 		(fields_autoplaced yes)
 		(effects
+			(font
+				(size 1.27 1.27)
+			)
+			(justify left bottom)
+		)
+	)
+	(label "TSAC.HVS.GND"
+		(at 43.18 99.06 0)
+		(fields_autoplaced yes)
+		(effects
