File: Stag11/LOOM - LV BOX.kicad_sch (KiCad schematic)
At the start: 22 parts

Commit message: Initial TSAL + Latching changes
Parts:
- removed Conn50: Molex_6x1P_Horizontal_THT, symbol Connectors_SUFST:Molex_6x1P_Horizontal_THT
- removed Conn52, Conn55: Molex_2x2P_Horizontal, symbol Connectors_SUFST:Molex_2x2P_Horizontal
- removed Conn71: Deutsch_DTM_12S_Pin, symbol Connectors_SUFST:Deutsch_DTM_12S_Pin
- added Conn75, Conn76, Conn77, Conn78, Conn79, Conn80, Conn81, Conn82, Conn83, Conn84, Conn85, Conn86: Molex_2x1S_Recepticle, symbol Connectors_SUFST:Molex_2x1S_Recepticle
- added Conn87: Molex_4x1S_Recepticle, symbol Connectors_SUFST:Molex_4x1S_Recepticle
Connections:
- net PCHG.AUX.EXC is gone; now on net CAN.S.HIGH: Conn61.27
- net SHUT.LATCHING is gone; now on net CANNODE.HVS.SIG: Conn60.3, Conn61.1
- net SHUT.TSMS is gone; now on net CANNODE.HVS.SIG: Conn60.4, Conn61.34
- net TS.DETECTED is gone; now on net CANNODE.HVS.SIG: Conn56.1, Conn62.1
- net TS.ON is gone; now on net CANNODE.HVS.SIG: Conn44.3, Conn61.16
- net TS.READY is gone; now on net CANNODE.HVS.SIG: Conn42.5, Conn61.9
- net CAN.S.HIGH: now also Conn87.3; no longer Conn46.2, Conn61.17, Conn61.18
- net CANNODE.HVS.SIG: now reaches Conn61.15
- net CANNODE.HVS.SIG: now also Conn62.4, Conn80.2, Conn81.2, Conn82.2, Conn83.2, Conn84.2, Conn85.2, Conn86.2
- net +AIR.AUX.EXC renamed CAN.NODE.GND
- net CAN.NODE.GND: now also Conn87.2
- net +AIR.AUX.GND: no longer names the net of Conn61.29
- net -AIR.AUX.EXC renamed CAN.NODE.EXC
- net CAN.NODE.EXC: now also Conn87.1
- net -AIR.AUX.GND renamed CAN.S.LOW
- net CAN.S.LOW: now also Conn46.2, Conn87.4
- net PCHG.AUX.GND: no longer names the net of Conn61.30
- no-connect marks 29 -> 27
Other:
- note added: "CAN-NODE"
- note added: "CURRENT.SENSE.SIG"
- note added: "PWR and DATA"
- note added: "SHUT.LATCHING"
- note added: "SHUT.TSMS"
- note added: "TS.DETECTED.HVBOX"
- note added: "TS.ON"
- note added: "TS.READY ?????"
- note added: "Temperature 1"
- note added: "Temperature 2"
- note added: "VCU.FAULT"
- note added: "Voltage 1"
- note added: "Voltage 10"
- note added: "Voltage 2"
- note added: "Voltage 3"
- note added: "Voltage 4"
- note added: "Voltage 5"
- note added: "Voltage 6"
- note added: "Voltage 7"
- note added: "Voltage 8"
- note added: "Voltage 9"
- note added: "~{GREEN.LED.ON}"

Commit message: Loom review. Couple of fixes and TODO lists added
Connections:
- net BATT+: no longer Conn51.2, Conn61.6
- net BMS.LED.GND: no longer Conn48.7, Conn48.8, Conn61.37, Conn61.38
- new net BATT-: Conn51.2, Conn61.6
- new net R2D.LED.GND: Conn48.8, Conn61.38
- new net TS.ON.LED.GND: Conn48.7, Conn61.37
Other:
- note added: "TODO: Dash excitations, needed or no? Dash soft reset Maybe combine some EXC signals, not sure"
Changed lines of the file:
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@@
 	(wire
 		(pts
-			(xy 457.2 78.74) (xy 457.2 323.85)
+			(xy 307.34 116.84) (xy 307.34 363.22)
 		)
 		(stroke
@@
 	(wire
 		(pts
-			(xy 307.34 116.84) (xy 307.34 363.22)
+			(xy 55.88 99.06) (xy 83.82 99.06)
 		)
 		(stroke
@@
 	(wire
 		(pts
-			(xy 55.88 99.06) (xy 83.82 99.06)
+			(xy 55.88 285.75) (xy 81.28 285.75)
 		)
 		(stroke
@@
 	(wire
 		(pts
-			(xy 55.88 285.75) (xy 81.28 285.75)
+			(xy 55.88 129.54) (xy 354.33 129.54)
 		)
 		(stroke
@@
 	(wire
 		(pts
-			(xy 346.71 43.18) (xy 55.88 43.18)
-		)
-		(stroke
-			(width 0)
-			(type default)
-		)
-	)
-	(wire
-		(pts
 			(xy 55.88 137.16) (xy 292.1 137.16)
 		)
@@
 	(wire
 		(pts
+			(xy 349.25 43.18) (xy 349.25 204.47)
+		)
+		(stroke
+			(width 0)
+			(type default)
+		)
+	)
+	(wire
+		(pts
 			(xy 351.79 132.08) (xy 351.79 160.02)
 		)
@@
 	(wire
 		(pts
+			(xy 55.88 127) (xy 356.87 127)
+		)
+		(stroke
+			(width 0)
+			(type default)
+		)
+	)
+	(wire
+		(pts
 			(xy 454.66 58.42) (xy 527.05 58.42)
 		)
@@
 	(wire
 		(pts
-			(xy 346.71 43.18) (xy 346.71 207.01)
-		)
-		(stroke
-			(width 0)
-			(type default)
-		)
-	)
-	(wire
-		(pts
-			(xy 55.88 45.72) (xy 349.25 45.72)
+			(xy 55.88 45.72) (xy 346.71 45.72)
 		)
 		(stroke
@@
 	(wire
 		(pts
-			(xy 515.62 78.74) (xy 457.2 78.74)
-		)
-		(stroke
-			(width 0)
-			(type default)
-		)
-	)
-	(wire
-		(pts
 			(xy 412.75 58.42) (xy 55.88 58.42)
 		)
@@
 	(wire
 		(pts
-			(xy 354.33 129.54) (xy 55.88 129.54)
+			(xy 55.88 48.26) (xy 433.07 48.26)
 		)
 		(stroke
@@
 	(wire
 		(pts
-			(xy 55.88 48.26) (xy 433.07 48.26)
+			(xy 311.15 111.76) (xy 311.15 257.81)
 		)
 		(stroke
@@
 	(wire
 		(pts
-			(xy 311.15 111.76) (xy 311.15 257.81)
+			(xy 86.36 101.6) (xy 86.36 290.83)
 		)
 		(stroke
@@
 	(wire
 		(pts
-			(xy 86.36 101.6) (xy 86.36 290.83)
+			(xy 346.71 45.72) (xy 346.71 207.01)
 		)
 		(stroke
@@
 	(wire
 		(pts
-			(xy 55.88 127) (xy 356.87 127)
-		)
-		(stroke
-			(width 0)
-			(type default)
-		)
-	)
-	(wire
-		(pts
-			(xy 349.25 45.72) (xy 349.25 204.47)
-		)
-		(stroke
-			(width 0)
-			(type default)
-		)
-	)
-	(wire
-		(pts
 			(xy 454.66 326.39) (xy 454.66 58.42)
 		)
@@
 	(wire
 		(pts
-			(xy 457.2 323.85) (xy 530.86 323.85)
-		)
-		(stroke
-			(width 0)
-			(type default)
-		)
-	)
-	(wire
-		(pts
 			(xy 367.03 114.3) (xy 55.88 114.3)
 		)
@@
 		)
 	)
+	(wire
+		(pts
+			(xy 55.88 43.18) (xy 349.25 43.18)
+		)
+		(stroke
+			(width 0)
+			(type default)
+		)
+	)
 	(rectangle
 		(start 29.845 278.13)
@@
 		)
 	)
+	(text "TODO:\nDash excitations, needed or no?\nDash soft reset\nMaybe combine some EXC signals, not sure\n"
+		(exclude_from_sim no)
+		(at 134.62 368.046 0)
+		(effects
+			(font
+				(size 3 3)
+				(bold yes)
+				(color 255 0 0 1)
+			)
+			(justify left bottom)
+		)
+	)
 	(text "SHUT.LATCHING\n"
 		(exclude_from_sim no)
@@
 		)
 	)
-	(text "VCU.FAULT"
-		(exclude_from_sim no)
-		(at 510.54 77.978 0)
-		(effects
-			(font
-				(size 1.27 1.27)
-			)
-		)
-	)
 	(text "TSAL"
 		(exclude_from_sim no)
@@
 	)
 	(label "R2D.LED.GND"
-		(at 57.15 129.54 0)
+		(at 57.15 127 0)
 		(fields_autoplaced yes)
 		(effects
@@
 		)
 	)
-	(label "TS.ON.LED.GND"
-		(at 57.15 127 0)
+	(label "BMS.LED.GND"
+		(at 57.15 129.54 0)
 		(fields_autoplaced yes)
 		(effects
@@
 	)
 	(label "BATT+"
-		(at 57.15 43.18 0)
+		(at 59.69 43.18 0)
 		(fields_autoplaced yes)
 		(effects
@@
 		)
 	)
+	(sheet_instances
+		(path "/"
+			(page "1")
+		)
+	)

Commit message: updates
Connections:
- net CANNODE.HVS.SIG: no longer Conn42.5, Conn44.3, Conn56.1, Conn60.3, Conn60.4, Conn61.1, Conn61.15, Conn61.16, Conn61.34, Conn61.9, Conn62.1, Conn80.2, Conn81.2, Conn82.2, Conn83.2, Conn85.2, Conn86.2
- net TS.DETECTED: now reaches Conn61.17
- net TS.DETECTED: now also Conn56.1, Conn62.1, Conn83.2
- net BMS.LED.GND renamed BMS.LED.K
- net IMD.LED.GND renamed IMD.LED.K
- net R2D.LED.GND renamed R2D.LED.K
- net TS.ON.LED.GND renamed TS.ON.LED.K
- net TSAL.GREEN.DASH.LED.GND renamed TSAL.GREEN.DASH.LED.K
- net TSAL.GREEN.LED.GND renamed TSAL.GREEN.LED.K
- net TSAL.RED.DASH.LED.GND renamed TSAL.RED.DASH.LED.K
- net TSAL.RED.LED.GND renamed TSAL.RED.LED.K
- new net SHUT.LATCHING: Conn60.3, Conn61.1, Conn86.2
- new net SHUT.TSMS: Conn60.4, Conn61.34, Conn85.2
- new net TS.ON: Conn44.3, Conn61.16, Conn81.2
- new net TS.READY: Conn42.5, Conn61.9, Conn80.2
- new net VOLTAGE.~{GREEN.LED.ON}.SIG: Conn61.15, Conn82.2
Other:
- note removed: "CURRENT.SENSE.SIG"
- note removed: "SHUT.LATCHING"
- note removed: "SHUT.TSMS"
- note removed: "TS.DETECTED.HVBOX"
- note removed: "TS.ON"
- note removed: "TS.READY ?????"
- note removed: "~{GREEN.LED.ON}"
Changed lines of the file:
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@@
 	)
 	(junction
+		(at 113.03 176.53)
+		(diameter 0)
+		(color 0 0 0 0)
+	)
+	(junction
 		(at 110.49 53.34)
 		(diameter 0)
@@
 	(wire
 		(pts
+			(xy 113.03 176.53) (xy 181.61 176.53)
+		)
+		(stroke
+			(width 0)
+			(type default)
+		)
+	)
+	(wire
+		(pts
 			(xy 313.69 109.22) (xy 55.88 109.22)
 		)
@@
 	(wire
 		(pts
+			(xy 113.03 176.53) (xy 113.03 73.66)
+		)
+		(stroke
+			(width 0)
+			(type default)
+		)
+	)
+	(wire
+		(pts
 			(xy 364.49 119.38) (xy 55.88 119.38)
 		)
@@
 	(wire
 		(pts
-			(xy 102.87 176.53) (xy 181.61 176.53)
+			(xy 102.87 176.53) (xy 113.03 176.53)
 		)
 		(stroke
@@
 	(wire
 		(pts
+			(xy 55.88 73.66) (xy 113.03 73.66)
+		)
+		(stroke
+			(width 0)
+			(type default)
+		)
+	)
+	(wire
+		(pts
 			(xy 454.66 326.39) (xy 454.66 58.42)
 		)
@@
 		)
 	)
-	(text "TS.READY ?????\n"
-		(exclude_from_sim no)
-		(at 80.518 331.724 0)
-		(effects
-			(font
-				(size 1.27 1.27)
-			)
-		)
-	)
 	(text "TODO:\nDash excitations, needed or no?\nDash soft reset\nMaybe combine some EXC signals, not sure\n"
 		(exclude_from_sim no)
@@
 		)
 	)
-	(text "SHUT.LATCHING\n"
-		(exclude_from_sim no)
-		(at 79.248 293.878 0)
-		(effects
-			(font
-				(size 1.27 1.27)
-			)
-		)
-	)
 	(text "Voltage 9"
 		(exclude_from_sim no)
@@
 		)
 	)
-	(text "TS.DETECTED.HVBOX"
-		(exclude_from_sim no)
-		(at 81.534 312.928 0)
-		(effects
-			(font
-				(size 1.27 1.27)
-			)
-		)
-	)
 	(text "Voltage 6"
 		(exclude_from_sim no)
@@
 		)
 	)
-	(text "TS.ON\n"
-		(exclude_from_sim no)
-		(at 75.438 325.628 0)
-		(effects
-			(font
-				(size 1.27 1.27)
-			)
-		)
-	)
 	(text "Voltage 5"
 		(exclude_from_sim no)
@@
 		)
 	)
-	(text "SHUT.TSMS"
-		(exclude_from_sim no)
-		(at 77.47 300.228 0)
-		(effects
-			(font
-				(size 1.27 1.27)
-			)
-		)
-	)
 	(text "Voltage 3"
 		(exclude_from_sim no)
@@
 		)
 	)
-	(text "CURRENT.SENSE.SIG\n"
-		(exclude_from_sim no)
-		(at 81.788 306.578 0)
-		(effects
-			(font
-				(size 1.27 1.27)
-			)
-		)
-	)
 	(text "Voltage 8"
 		(exclude_from_sim no)
@@
 		)
 	)
-	(text "~{GREEN.LED.ON}\n"
-		(exclude_from_sim no)
-		(at 78.994 319.278 0)
-		(effects
-			(font
-				(size 1.27 1.27)
-			)
-		)
-	)
 	(text "Voltage 1"
 		(exclude_from_sim no)
@@
 		)
 	)
-	(label "TSAL.GREEN.LED.GND"
+	(label "TSAL.GREEN.LED.K"
 		(at 530.86 271.78 180)
 		(fields_autoplaced yes)
@@
 		)
 	)
-	(label "R2D.LED.GND"
+	(label "R2D.LED.K"
 		(at 57.15 127 0)
 		(fields_autoplaced yes)
@@
 		)
 	)
-	(label "TSAL.GREEN.LED.GND"
+	(label "TSAL.GREEN.LED.K"
 		(at 57.15 63.5 0)
 		(fields_autoplaced yes)
@@
 		)
 	)
-	(label "BMS.LED.GND"
+	(label "BMS.LED.K"
 		(at 57.15 129.54 0)
 		(fields_autoplaced yes)
@@
 		)
 	)
-	(label "VOLTAGE.SIG"
+	(label "VOLTAGE.SHUT.LATCHING.SIG"
 		(at 58.42 294.64 0)
 		(fields_autoplaced yes)
@@
 		)
 	)
-	(label "TS.ON.LED.GND"
+	(label "TS.ON.LED.K"
 		(at 57.15 124.46 0)
 		(fields_autoplaced yes)
@@
 		)
 	)
-	(label "VOLTAGE.SIG"
+	(label "VOLTAGE.TS.DETECTED.SIG"
 		(at 58.42 313.69 0)
 		(fields_autoplaced yes)
@@
 		)
 	)
-	(label "TSAL.RED.DASH.LED.GND"
+	(label "TSAL.RED.DASH.LED.K"
 		(at 530.86 279.4 180)
 		(fields_autoplaced yes)
@@
 		)
 	)
-	(label "R2D.LED.GND"
+	(label "R2D.LED.K"
 		(at 527.05 154.94 180)
 		(fields_autoplaced yes)
@@
 		)
 	)
-	(label "TSAL.RED.LED.GND"
+	(label "TSAL.RED.LED.K"
 		(at 530.86 274.32 180)
 		(fields_autoplaced yes)
@@
 		)
 	)
-	(label "VOLTAGE.SIG"
+	(label "VOLTAGE.TS.READY.SIG"
 		(at 58.42 332.74 0)
 		(fields_autoplaced yes)
@@
 		)
 	)
-	(label "BMS.LED.GND"
+	(label "BMS.LED.K"
 		(at 527.05 157.48 180)
 		(fields_autoplaced yes)
@@
 		)
 	)
-	(label "TSAL.GREEN.DASH.LED.GND"
+	(label "TSAL.GREEN.DASH.LED.K"
 		(at 57.15 55.88 0)
 		(fields_autoplaced yes)
@@
 		)
 	)
-	(label "IMD.LED.GND"
+	(label "IMD.LED.K"
 		(at 57.15 132.08 0)
 		(fields_autoplaced yes)
@@
 		)
 	)
-	(label "TSAL.GREEN.DASH.LED.GND"
+	(label "TSAL.GREEN.DASH.LED.K"
 		(at 530.86 276.86 180)
 		(fields_autoplaced yes)
@@
 		)
 	)
+	(label "TS.DETECTED.DASH.SPLICE"
+		(at 57.15 73.66 0)
+		(fields_autoplaced yes)
+		(effects
+			(font
+				(size 1.27 1.27)
+			)
+			(justify left bottom)
+		)
+	)
 	(label "LATCHING.EXC"
 		(at 530.86 355.6 180)
@@
 		)
 	)
-	(label "VOLTAGE.SIG"
+	(label "VOLTAGE.TS.ON.SIG"
 		(at 58.42 326.39 0)
 		(fields_autoplaced yes)
@@
 		)
 	)
-	(label "VOLTAGE.SIG"
+	(label "VOLTAGE.SHUT.TSMS.SIG"
 		(at 58.42 300.99 0)
 		(fields_autoplaced yes)
@@
 		)
 	)
-	(label "TS.ON.LED.GND"
+	(label "TS.ON.LED.K"
 		(at 527.05 152.4 180)
 		(fields_autoplaced yes)
@@
 	)
 	(label "BATT+"
-		(at 59.69 43.18 0)
+		(at 57.15 43.18 0)
 		(fields_autoplaced yes)
 		(effects
@@
 		)
 	)
-	(label "VOLTAGE.SIG"
+	(label "VOLTAGE.CURRENT.SENSE.SIG"
 		(at 58.42 307.34 0)
 		(fields_autoplaced yes)
@@
 		)
 	)
-	(label "VOLTAGE.SIG"
+	(label "VOLTAGE.~{GREEN.LED.ON}.SIG"
 		(at 58.42 320.04 0)
 		(fields_autoplaced yes)
@@
 		)
 	)
-	(label "TSAL.RED.LED.GND"
+	(label "TSAL.RED.LED.K"
 		(at 57.15 60.96 0)
 		(fields_autoplaced yes)
@@
 		)
 	)
-	(label "IMD.LED.GND"
+	(label "IMD.LED.K"
 		(at 527.05 160.02 180)
 		(fields_autoplaced yes)

Commit message: Front and Rear almost complete
TODO: Arrange power
Parts:
- added Conn55: Molex_2x2P_Horizontal, symbol Connectors_SUFST:Molex_2x2P_Horizontal
Connections:
- net SAGL.SIG: now also Conn79.2
- net TS.ON.LED.K: no longer Conn61.37
- net TSAC.HVS.EXC: now reaches Conn61.29
- net TSAC.HVS.EXC: now also Conn55.3
- net TSAC.HVS.GND: now reaches Conn61.30
- net TSAC.HVS.GND: now also Conn55.4
- net VOLTAGE.~{GREEN.LED.ON}.SIG renamed TSAL.GREEN.LIGHT
- no-connect marks 27 -> 30
Other:
- note added: "-->"
- note added: "Splice to CAN node"

Commit message: I forgot what I did but changed CAN layout
Connections:
- net CAN.NODE.EXC: no longer Conn61.25
- net CAN.NODE.GND: no longer Conn61.26
- net CAN.S.HIGH: now also Conn61.25
- net CAN.S.LOW: now also Conn61.26
- net VOLTAGE.SHUT.TSAC.INTERLOCK.SIG: now reaches Conn61.18
- net VOLTAGE.SHUT.TSAC.INTERLOCK.SIG: now also Conn78.2
Other:
- note added: "<--"
- note added: "Splice to CAN node and VCU"
- note added: "TSAL + Latching and CANnode can combine to free up 2 pins if required"
- note removed: "Splice to CAN node"
Changed lines of the file:
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@@
 	(paper "A2")
 	(junction
+		(at 91.44 99.06)
+		(diameter 0)
+		(color 0 0 0 0)
+	)
+	(junction
 		(at 105.41 68.58)
 		(diameter 0)
@@
 	)
 	(junction
+		(at 88.9 101.6)
+		(diameter 0)
+		(color 0 0 0 0)
+	)
+	(junction
 		(at 110.49 53.34)
 		(diameter 0)
@@
 	(wire
 		(pts
-			(xy 55.88 96.52) (xy 81.28 96.52)
+			(xy 294.64 334.01) (xy 294.64 134.62)
 		)
 		(stroke
@@
 	(wire
 		(pts
-			(xy 294.64 334.01) (xy 294.64 134.62)
+			(xy 284.48 347.98) (xy 284.48 144.78)
 		)
 		(stroke
@@
 	(wire
 		(pts
-			(xy 284.48 347.98) (xy 284.48 144.78)
+			(xy 91.44 99.06) (xy 91.44 93.98)
+		)
+		(stroke
+			(width 0)
+			(type default)
+			(color 0 0 255 1)
+		)
+	)
+	(wire
+		(pts
+			(xy 81.28 238.76) (xy 81.28 285.75)
 		)
 		(stroke
@@
 	(wire
 		(pts
-			(xy 83.82 99.06) (xy 381 99.06)
+			(xy 83.82 99.06) (xy 91.44 99.06)
 		)
 		(stroke
@@
 	(wire
 		(pts
+			(xy 88.9 96.52) (xy 55.88 96.52)
+		)
+		(stroke
+			(width 0)
+			(type default)
+			(color 0 0 255 1)
+		)
+	)
+	(wire
+		(pts
 			(xy 349.25 204.47) (xy 530.86 204.47)
 		)
@@
 	(wire
 		(pts
+			(xy 118.11 76.2) (xy 55.88 76.2)
+		)
+		(stroke
+			(width 0)
+			(type default)
+			(color 155 0 0 1)
+		)
+	)
+	(wire
+		(pts
 			(xy 373.38 114.3) (xy 527.05 114.3)
 		)
@@
 			(width 0)
 			(type default)
-			(color 255 0 0 1)
+			(color 155 0 0 1)
 		)
 	)
@@
 	(wire
 		(pts
-			(xy 55.88 93.98) (xy 78.74 93.98)
-		)
-		(stroke
-			(width 0)
-			(type default)
-		)
-	)
-	(wire
-		(pts
 			(xy 378.46 109.22) (xy 527.05 109.22)
 		)
@@
 	(wire
 		(pts
+			(xy 55.88 345.44) (xy 118.11 345.44)
+		)
+		(stroke
+			(width 0)
+			(type default)
+			(color 155 0 0 1)
+		)
+	)
+	(wire
+		(pts
 			(xy 351.79 160.02) (xy 528.32 160.02)
 		)
@@
 	(wire
 		(pts
-			(xy 86.36 101.6) (xy 378.46 101.6)
+			(xy 88.9 101.6) (xy 378.46 101.6)
+		)
+		(stroke
+			(width 0)
+			(type default)
+			(color 0 0 255 1)
+		)
+	)
+	(wire
+		(pts
+			(xy 86.36 101.6) (xy 88.9 101.6)
 		)
 		(stroke
@@
 			(width 0)
 			(type default)
-			(color 255 0 0 1)
+			(color 155 0 0 1)
 		)
 	)
@@
 	(wire
 		(pts
-			(xy 81.28 96.52) (xy 81.28 285.75)
-		)
-		(stroke
-			(width 0)
-			(type default)
-		)
-	)
-	(wire
-		(pts
 			(xy 530.86 312.42) (xy 179.07 312.42)
 		)
@@
 	(wire
 		(pts
-			(xy 78.74 93.98) (xy 78.74 283.21)
+			(xy 284.48 144.78) (xy 55.88 144.78)
 		)
 		(stroke
@@
 	(wire
 		(pts
-			(xy 284.48 144.78) (xy 55.88 144.78)
+			(xy 55.88 307.34) (xy 100.33 307.34)
 		)
 		(stroke
@@
 	(wire
 		(pts
-			(xy 55.88 307.34) (xy 100.33 307.34)
+			(xy 378.46 86.36) (xy 378.46 93.98)
 		)
 		(stroke
@@
 	(wire
 		(pts
-			(xy 378.46 86.36) (xy 378.46 93.98)
+			(xy 527.05 55.88) (xy 452.12 55.88)
 		)
 		(stroke
@@
 	(wire
 		(pts
-			(xy 527.05 55.88) (xy 452.12 55.88)
+			(xy 332.74 91.44) (xy 332.74 212.09)
 		)
 		(stroke
@@
 	(wire
 		(pts
-			(xy 332.74 91.44) (xy 332.74 212.09)
+			(xy 316.23 297.18) (xy 530.86 297.18)
 		)
 		(stroke
@@
 	(wire
 		(pts
-			(xy 316.23 297.18) (xy 530.86 297.18)
+			(xy 55.88 132.08) (xy 351.79 132.08)
 		)
 		(stroke
@@
 	(wire
 		(pts
-			(xy 55.88 132.08) (xy 351.79 132.08)
+			(xy 55.88 93.98) (xy 91.44 93.98)
 		)
 		(stroke
 			(width 0)
 			(type default)
+			(color 0 0 255 1)
 		)
 	)
@@
 			(width 0)
 			(type default)
-			(color 255 0 0 1)
+			(color 155 0 0 1)
 		)
 	)
@@
 	(wire
 		(pts
+			(xy 91.44 99.06) (xy 381 99.06)
+		)
+		(stroke
+			(width 0)
+			(type default)
+			(color 0 0 255 1)
+		)
+	)
+	(wire
+		(pts
 			(xy 361.95 144.78) (xy 528.32 144.78)
 		)
@@
 			(width 0)
 			(type default)
-			(color 255 0 0 1)
+			(color 155 0 0 1)
 		)
 	)
@@
 	(wire
 		(pts
+			(xy 78.74 238.76) (xy 78.74 283.21)
+		)
+		(stroke
+			(width 0)
+			(type default)
+		)
+	)
+	(wire
+		(pts
 			(xy 367.03 114.3) (xy 55.88 114.3)
 		)
@@
 	(wire
 		(pts
+			(xy 118.11 345.44) (xy 118.11 76.2)
+		)
+		(stroke
+			(width 0)
+			(type default)
+			(color 155 0 0 1)
+		)
+	)
+	(wire
+		(pts
 			(xy 528.32 139.7) (xy 364.49 139.7)
 		)
@@
 	(wire
 		(pts
+			(xy 88.9 101.6) (xy 88.9 96.52)
+		)
+		(stroke
+			(width 0)
+			(type default)
+			(color 0 0 255 1)
+		)
+	)
+	(wire
+		(pts
 			(xy 335.28 209.55) (xy 335.28 88.9)
 		)
@@
 		)
 	)
-	(text "Splice to CAN node\n"
+	(text "Splice to CAN node and VCU\n\n"
 		(exclude_from_sim no)
-		(at 84.074 96.52 0)
+		(at 82.804 99.06 0)
 		(effects
 			(font
@@
 	(text "-->\n"
 		(exclude_from_sim no)
-		(at 91.694 100.584 0)
+		(at 70.104 100.584 0)
 		(effects
 			(font
@@
 		)
 	)
+	(text "TSAL + Latching and CANnode can combine \nto free up 2 pins if required"
+		(exclude_from_sim no)
+		(at 48.26 154.178 0)
+		(effects
+			(font
+				(size 1.27 1.27)
+			)
+		)
+	)
 	(text "Voltage 8"
 		(exclude_from_sim no)
@@
 		)
 	)
+	(text "<--\n"
+		(exclude_from_sim no)
+		(at 70.104 95.504 0)
+		(effects
+			(font
+				(size 1.27 1.27)
+			)
+		)
+	)
 	(text "Voltage 10"
 		(exclude_from_sim no)
@@
 		)
 	)
-	(label "CAN.NODE.EXC"
-		(at 57.15 93.98 0)
-		(fields_autoplaced yes)
-		(effects
-			(font
-				(size 1.27 1.27)
-			)
-			(justify left bottom)
-		)
-	)
 	(label "TSAL.RESET+"
 		(at 57.15 111.76 0)
@@
 		)
 	)
+	(label "CAN.S.HIGH"
+		(at 57.15 93.98 0)
+		(fields_autoplaced yes)
+		(effects
+			(font
+				(size 1.27 1.27)
+			)
+			(justify left bottom)
+		)
+	)
 	(label "TSAC.HVS.GND"
 		(at 57.15 106.68 0)
@@
 		)
 	)
+	(label "CAN.S.LOW"
+		(at 57.15 96.52 0)
+		(fields_autoplaced yes)
+		(effects
+			(font
+				(size 1.27 1.27)
+			)
+			(justify left bottom)
+		)
+	)
 	(label "CAN.NODE.EXC"
 		(at 58.42 283.21 0)
@@
 		)
 	)
-	(label "CAN.NODE.GND"
-		(at 57.15 96.52 0)
-		(fields_autoplaced yes)
-		(effects
-			(font
-				(size 1.27 1.27)
-			)
-			(justify left bottom)
-		)
-	)
 	(label "VOLTAGE.GND"
 		(at 58.42 303.53 0)
@@
 		)
 	)
-	(label "VOLTAGE.SIG"
+	(label "VOLTAGE.SHUT.TSAC.INTERLOCK.SIG"
 		(at 58.42 345.44 0)
 		(fields_autoplaced yes)
@@
 		)
 	)
+	(label "VOLTAGE.SHUT.TSAC.INTERLOCK.SIG"
+		(at 57.15 76.2 0)
+		(fields_autoplaced yes)
+		(effects
+			(font
+				(size 1.27 1.27)
+			)
+			(justify left bottom)
+		)
+	)

Commit message: Added power splice to LV box, connected PDM to CAN
Connections:
- net VCU.EXC is gone; now on net CAN.NODE.EXC: Conn47.1, Conn61.4
- net BATT+: now also Conn61.46; no longer Conn61.5
- net BATT-: now also Conn61.47; no longer Conn61.6
- net CAN.NODE.EXC: now also Conn51.3, Conn60.1
- net CAN.NODE.GND: now also Conn47.2, Conn51.4, Conn60.2, Conn61.5
- removed net LATCHING.EXC: Conn60.1, Conn61.46
- removed net LATCHING.GND: Conn60.2, Conn61.47
- net TSAL.EXC: no longer names the net of Conn61.23
- net TSAL.EXC: no longer Conn51.3
- net TSAL.GND: no longer names the net of Conn61.24
- net TSAL.GND: no longer Conn51.4
- net VCU.GND: no longer names the net of Conn61.14
- net VCU.GND: no longer Conn47.2
