File: Stag11/LOOM - LV BOX.kicad_sch (KiCad schematic)
At the start: 32 parts

Commit message: Reordered shutdown loop and spliced power in LV box
Parts:
- added Conn88: TODO: CHECK CONNECTOR, symbol Connectors_SUFST:Current Sensor Connector
Connections:
- net VCU.UART.TX: now reaches Conn61.23
- net VCU.UART.RX: now reaches Conn61.24
- net SHUT.TSMS renamed SHUT.HVD.INTERLOCK
Changed lines of the file:
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@@
 	(wire
 		(pts
+			(xy 370.84 96.52) (xy 487.68 96.52)
+		)
+		(stroke
+			(width 0)
+			(type default)
+		)
+	)
+	(wire
+		(pts
 			(xy 88.9 96.52) (xy 55.88 96.52)
 		)
@@
 	(wire
 		(pts
+			(xy 55.88 91.44) (xy 370.84 91.44)
+		)
+		(stroke
+			(width 0)
+			(type default)
+		)
+	)
+	(wire
+		(pts
 			(xy 55.88 285.75) (xy 81.28 285.75)
 		)
@@
 	(wire
 		(pts
+			(xy 485.14 88.9) (xy 485.14 86.36)
+		)
+		(stroke
+			(width 0)
+			(type default)
+		)
+	)
+	(wire
+		(pts
+			(xy 487.68 96.52) (xy 487.68 88.9)
+		)
+		(stroke
+			(width 0)
+			(type default)
+		)
+	)
+	(wire
+		(pts
 			(xy 55.88 129.54) (xy 354.33 129.54)
 		)
@@
 	(wire
 		(pts
+			(xy 55.88 88.9) (xy 485.14 88.9)
+		)
+		(stroke
+			(width 0)
+			(type default)
+		)
+	)
+	(wire
+		(pts
+			(xy 370.84 91.44) (xy 370.84 96.52)
+		)
+		(stroke
+			(width 0)
+			(type default)
+		)
+	)
+	(wire
+		(pts
 			(xy 55.88 137.16) (xy 292.1 137.16)
 		)
@@
 	(wire
 		(pts
+			(xy 487.68 88.9) (xy 504.19 88.9)
+		)
+		(stroke
+			(width 0)
+			(type default)
+		)
+	)
+	(wire
+		(pts
 			(xy 530.86 307.34) (xy 181.61 307.34)
 		)
@@
 	(wire
 		(pts
+			(xy 485.14 86.36) (xy 504.19 86.36)
+		)
+		(stroke
+			(width 0)
+			(type default)
+		)
+	)
+	(wire
+		(pts
 			(xy 500.38 212.09) (xy 530.86 212.09)
 		)
@@
 		)
 	)
-	(label "SHUT.TSMS"
-		(at 57.15 116.84 0)
-		(fields_autoplaced yes)
-		(effects
-			(font
-				(size 1.27 1.27)
-			)
-			(justify left bottom)
-		)
-	)
 	(label "PWR_SPLICE.EXC"
 		(at 57.15 40.64 0)
@@
 		)
 	)
+	(label "VCU.UART.TX"
+		(at 504.19 86.36 0)
+		(fields_autoplaced yes)
+		(effects
+			(font
+				(size 1.27 1.27)
+			)
+			(justify left bottom)
+		)
+	)
 	(label "TS.ON"
 		(at 57.15 71.12 0)
@@
 		)
 	)
+	(label "VCU.UART.RX"
+		(at 504.19 88.9 0)
+		(fields_autoplaced yes)
+		(effects
+			(font
+				(size 1.27 1.27)
+			)
+			(justify left bottom)
+		)
+	)
 	(label "SPARE.GND"
 		(at 525.78 81.28 180)
@@
 		)
 	)
+	(label "VCU.UART.TX"
+		(at 57.15 88.9 0)
+		(fields_autoplaced yes)
+		(effects
+			(font
+				(size 1.27 1.27)
+			)
+			(justify left bottom)
+		)
+	)
 	(label "LATCHING.GND"
 		(at 530.86 358.14 180)
@@
 		)
 	)
-	(label "SHUT.TSMS"
-		(at 530.86 363.22 180)
-		(fields_autoplaced yes)
-		(effects
-			(font
-				(size 1.27 1.27)
-			)
-			(justify right bottom)
-		)
-	)
 	(label "SPARE.EXC"
 		(at 525.78 76.2 180)
@@
 		)
 	)
+	(label "SHUT.HVD.INTERLOCK"
+		(at 57.15 116.84 0)
+		(fields_autoplaced yes)
+		(effects
+			(font
+				(size 1.27 1.27)
+			)
+			(justify left bottom)
+		)
+	)
 	(label "LATCHING.RESET-"
 		(at 57.15 137.16 0)
@@
 		)
 	)
+	(label "VCU.UART.RX"
+		(at 57.15 91.44 0)
+		(fields_autoplaced yes)
+		(effects
+			(font
+				(size 1.27 1.27)
+			)
+			(justify left bottom)
+		)
+	)
 	(label "BPS.SIG"
 		(at 57.15 48.26 0)
@@
 		)
 	)
-	(label "VOLTAGE.SHUT.TSMS.SIG"
+	(label "VOLTAGE.SHUT.HVD.INTERLOCK.SIG"
 		(at 58.42 300.99 0)
 		(fields_autoplaced yes)
@@
 		)
 	)
+	(label "SHUT.HVD.INTERLOCK"
+		(at 530.86 363.22 180)
+		(fields_autoplaced yes)
+		(effects
+			(font
+				(size 1.27 1.27)
+			)
+			(justify right bottom)
+		)
+	)
 	(label "PWR_SPLICE.GND"
 		(at 501.65 358.14 180)
@@
 		)
 	)
-	(hierarchical_label "Accumulator LV Connector"
-		(shape input)
-		(at 50.8 237.49 180)
-		(fields_autoplaced yes)
-		(effects
-			(font
-				(size 1.27 1.27)
-			)
-			(justify right)
-		)
-	)
 	(hierarchical_label "LV - HV Connector"
 		(shape input)
@@
 					(unit 1)
 				)
+			)
+		)
+	)
+	(symbol
+		(lib_id "Connectors_SUFST:Current Sensor Connector")
+		(at 55.88 214.63 0)
+		(unit 1)
+		(exclude_from_sim no)
+		(in_bom yes)
+		(on_board yes)
+		(dnp no)
+		(fields_autoplaced yes)
+		(property "Reference" "Conn88"
+			(at 53.6621 210.82 0)
+			(effects
+				(font
+					(size 1.27 1.27)
+				)
+			)
+		)
+		(property "Value" "TODO: CHECK CONNECTOR"
+			(at 53.6621 213.36 0)
+			(effects
+				(font
+					(size 1.27 1.27)
+				)
+			)
+		)
+		(property "Footprint" ""
+			(at 55.88 213.995 0)
+			(effects
+				(font
+					(size 1.27 1.27)
+				)
+				(hide yes)
+			)
+		)
+		(property "Datasheet" ""
+			(at 55.88 213.995 0)
+			(effects
+				(font
+					(size 1.27 1.27)
+				)
+				(hide yes)
+			)
+		)
+		(property "Description" ""
+			(at 55.88 214.63 0)
+			(effects
+				(font
+					(size 1.27 1.27)
+				)
+				(hide yes)
+			)
+		)
+		(property "P/N" "TYCO 1-1456426-5"
+			(at 52.07 217.8055 0)
+			(effects
+				(font
+					(size 1.27 1.27)
+				)
+				(justify right)
+				(hide yes)
+			)
+		)
+		(property "Conn Name" ""
+			(at 55.88 214.63 0)
+			(effects
+				(font
+					(size 1.27 1.27)
+				)
+			)
+		)
+		(pin "1"
+		)
+		(pin "2"
+		)
+		(pin "3"
+		)
+		(pin "4"
+		)
+		(instances
+			(project "Stag11"
+				(path "/03011643-0690-4b85-ab78-d6a62dae52b1/8b0beb0f-c453-4b15-89f4-ecc97c450520"
+					(reference "Conn88")
+					(unit 1)
+				)

Commit message: Added TSAL+LATCHING board
Parts:
- removed Conn51, Conn55, Conn56, Conn59, Conn60: Molex_2x2P_Horizontal, symbol Connectors_SUFST:Molex_2x2P_Horizontal
- removed Conn53, Conn57, Conn58: Molex_2x1P_Horizontal_THT, symbol Connectors_SUFST:Molex_2x1P_Horizontal_THT
- removed Conn54: Molex_6x1P_Horizontal_THT, symbol Connectors_SUFST:Molex_6x1P_Horizontal_THT
- added J10: LATCHING, Connector_Molex:Molex_Micro-Fit_3.0_43045-1200_2x06_P3.00mm_Horizontal, symbol Connector_Generic:Conn_01x12
- added J8: TSAL, Connector_Molex:Molex_Micro-Fit_3.0_43045-1200_2x06_P3.00mm_Horizontal, symbol Connector_Generic:Conn_01x12
- added J9: POWER, Connector_Molex:Molex_Micro-Fit_3.0_43045-1200_2x06_P3.00mm_Horizontal, symbol Connector_Generic:Conn_01x12
- Conn88: symbol Connectors_SUFST:Current Sensor Connector -> Connectors_SUFST:Deutsch_DTM_6P_Pin; P/N TYCO 1-1456426-5 -> DTM046P-E003
Connections:
- net BATT+: now also J8.12 (Pin_12)
- net BATT-: now also J8.6 (Pin_6)
- net BMS.FAULT.LATCHING: now also J10.2 (Pin_2)
- net CAN.NODE.EXC: now also J9.6 (Pin_6)
- net CAN.NODE.GND: now also J9.12 (Pin_12)
- net IMD.FAULT.LATCHING: now also J10.1 (Pin_1)
- net IMD.OK: now also J10.8 (Pin_8)
- net LATCHING.RESET+: now also J10.4 (Pin_4)
- net LATCHING.RESET-: now also J10.10 (Pin_10)
- net REB.HVS.EXC: now also J9.3 (Pin_3)
- net REB.HVS.GND: now also J9.9 (Pin_9)
- net SHUT.HVD.INTERLOCK: now also J10.11 (Pin_11), J10.5 (Pin_5)
- net SHUT.LATCHING: now also J10.12 (Pin_12), J10.6 (Pin_6)
- net TS.DETECTED: now also J8.9 (Pin_9)
- net TSAC.HVS.EXC: now also J9.2 (Pin_2)
- net TSAC.HVS.GND: now also J9.8 (Pin_8)
- net TSAL.GREEN.DASH.LED.K: now also J8.3 (Pin_3)
- net TSAL.GREEN.LIGHT: now also J8.11 (Pin_11)
- net TSAL.LED.EXC: now also J9.1 (Pin_1)
- net TSAL.RED.DASH.LED.K: now also J8.10 (Pin_10)
- net TSAL.RESET+: now also J8.8 (Pin_8)
- net TSAL.RESET-: now also J8.7 (Pin_7)
- net ~{BMS.DISCHARGE.ENABLE}: now also J10.7 (Pin_7)
- net TSAL.LED.GND: now reaches Conn61.14
- net TSAL.LED.GND: now also J9.7 (Pin_7)
- net BMS.FAULT renamed ~{BMS.FAULT}
- net ~{BMS.FAULT}: now also J10.9 (Pin_9)
- net TSAL.GREEN.LED.K renamed TSAL.GREEN.LED.EN
- net TSAL.GREEN.LED.EN: now also J8.4 (Pin_4)
- net TSAL.RED.LED.K renamed TSAL.RED.LED.EN
- net TSAL.RED.LED.EN: now also J8.5 (Pin_5)
- no-connect marks 30 -> 26
Other:
- note added: "TODO: CHECK IF IMD AND BMS GO TO DASH OR VCU"
- note added: "TODO: SPEC Connectors for programmer (5 pin)"
- note added: "TSAL + Latching"
- note removed: "LATCHING"
- note removed: "TODO: SPEC Connectors"
- note removed: "TSAL"
- note removed: "TSAL + Latching and CANnode can combine to free up 2 pins if required"
- note removed: "To be combined"
- note removed: "VCU.FAULT"
