File: Stag11/loom-accumulator.kicad_sch (KiCad schematic)
At the start: 47 parts, among them J3 Conn_01x12, J4 Conn_01x12, J5 ATM064S, J6 ATM064S, J7 ATM064S, M1 AIL FAN, SW7 EV200HAANA, SW8 EV200HAANA, SW9 GV222BAB

Commit message: Updated Accu Internal Wiring
Parts:
- removed Conn3: Deutsch_DTM_2P_Pin, symbol Connectors_SUFST:Deutsch_DTM_2P_Pin
- removed R2: 15, symbol Device:R_Small
- removed SegmentPower: Deutsch_DTM_6P_Pin, symbol Connectors_SUFST:Deutsch_DTM_6P_Pin
- added Conn54: AIL FAN, symbol Connector_Generic:Conn_01x04
- added SegmentPower: Deutsch_DTM_12P_Pin, symbol Connectors_SUFST:Deutsch_DTM_12P_Pin
- Conn2: symbol Connectors_SUFST:Deutsch_DTM_2S_Pin -> Connector_Generic:Conn_01x04; P/N DTM062S-E007 -> KK 254
- J3, J4: value Conn_01x12 -> Micro-Fit 02x06
- J5, J6: value ATM064S -> Micro-Fit 02x02
- XK1A: value Conn_01x08 -> MNL 01x08
Connections:
- net -AIR.AUX.GND is gone; now on net GND: J3.4 (Pin_4), J7.1 (Pin_1)
- net PCHG.AUX.GND is gone; now on net GND: J3.6 (Pin_6), J5.1 (Pin_1)
- net +AIR.AUX.EXC: now also J3.9 (Pin_9), J7.2 (Pin_2); no longer J3.10 (Pin_10), J6.2 (Pin_2)
- net +AIR.EXC: now also J4.12 (Pin_12), J7.4 (Pin_4); no longer J4.11 (Pin_11), J6.4 (Pin_4)
- net +AIR.GND: now also Conn2.1 (Pin_1), SegmentPower.10, SegmentPower.3; no longer Conn2.2
- net -AIR.AUX.EXC: now also J3.10 (Pin_10), J6.2 (Pin_2); no longer J3.9 (Pin_9), J7.2 (Pin_2)
- net -AIR.EXC: now also Conn?.17, J4.11 (Pin_11), J4.3 (Pin_3), J6.4 (Pin_4), SegmentSignals.8, SegmentSignals1.8; no longer J4.12 (Pin_12), J7.4 (Pin_4)
- net ACCU.EXC: now also Conn2.2 (Pin_2), SegmentPower.2
- net CHASSIS.GND: now also SegmentPower.6, SegmentPower.7
- net SHDN_IN: no longer Conn?.17, SegmentSignals.8, SegmentSignals1.8
- net SHUT.IN: now also SegmentPower.1, SegmentPower.12
- net TSAC.HVS.EXC: now also SegmentPower.4
- net TSAC.HVS.GND: now also SegmentPower.5
- net at M1.1 (+): now also Conn54.2 (Pin_2)
- net at M1.2 (-): now also Conn54.1 (Pin_1)
- net NC_KEY: now reaches J3.12 (Pin_12)
- net NC_KEY: now also J4.6 (Pin_6)
- net +AIR.AUX.GND renamed GND
- no-connect marks 58 -> 67
Other:
- note added: "Modification on TRC PCB connects P11 to P06 with wire on back"
- note added: "Note: NC keyed sockets removed on connector housing; Header pins filled with epoxy"
- note removed: "ATM"
- note removed: "Panel Mount"
- moved on the sheet: DCLINK, HV+, HV-, PWR, SIGNALS

Commit message: Added BMS charge power replacing the redundant SHUT.IN pin.
Connections:
- net ACCU.EXC: no longer CONN?.3 (Pin_3)
- net SHUT.IN: no longer Conn?.34
- new net ACCU.CHARGE.EXC: CONN?.3 (Pin_3), Conn?.34
