File: Stag11/loom-roll-hoop.kicad_sch (KiCad schematic)
At the start: 5 parts

Commit message: Fixed mislabelled wires for precharge
Changed lines of the file:
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@@
 (kicad_sch
-	(version 20231120)
+	(version 20250114)
 	(generator "eeschema")
-	(generator_version "8.0")
+	(generator_version "9.0")
 	(paper "A4")
 	(title_block
