File: Stag12/loom-roll-hoop.kicad_sch (KiCad schematic)
At the start: 5 parts

Commit message: Started rear loom
Parts:
- removed Conn?: Deutsch_DTM_2P_Pin, symbol Connectors_SUFST:Deutsch_DTM_2P_Pin
- removed Conn? (x2): Deutsch_DTM_2S_Pin, symbol Connectors_SUFST:Deutsch_DTM_2S_Pin
- removed Conn?: Deutsch_DTM_6S_Pin, symbol Connectors_SUFST:Deutsch_DTM_6S_Pin
- removed Conn?: Deutsch_DTM_6P_Pin, symbol Connectors_SUFST:Deutsch_DTM_6P_Pin
Connections:
- no-connect marks 2 -> 0
