File: Stag12/acronyms.kicad_sch (KiCad schematic)
At the start: 0 parts

Commit message: just moved can-bus to acronyms doc so i dont have to keep switching branches - thanks anna
Parts:
- added J100, J101, J102 (x2), J103, J104, J105 (x2), J106 (x2), J107, J108, J109, J110 (x2), J111 (x2), J112, J113, J114, J115, J116 (x2), J117, J118, J119, J120, J121, J122, J123, J124, J126, J127, J128, J129, J130, J131, J138, J157, J159, J160, J161, J163, J169, J178, J180, J227, J228, J229, J231, J233, J234, J236, J237, J239, J240, J247, J90, J97 (x2), J98, J99 (x2): Conn_02x02_Counter_Clockwise, symbol Connector_Generic:Conn_02x02_Counter_Clockwise
- added J101, J104, J107, J108, J109, J113, J114, J115, J118, J119, J120, J121, J122, J123, J158, J164, J165, J170, J173, J174, J182, J217, J230, J235, J238, J242, J243, J244, J245, J246, J248, J90: Conn_01x02, symbol Connector_Generic:Conn_01x02
- added J117, J136, J177, J181: Conn_01x05, symbol Connector_Generic:Conn_01x05
- added J132, J137, J232, J241: Conn_01x03, symbol Connector_Generic:Conn_01x03
- added J133, J135, J168, J179: Conn_01x04, symbol Connector_Generic:Conn_01x04
- added J98: Conn_02x04_Counter_Clockwise, symbol Connector_Generic:Conn_02x04_Counter_Clockwise
Connections:
- new net: J169.1 (Pin_1), J169.2 (Pin_2)
- new net: J169.3 (Pin_3), J169.4 (Pin_4)
- new net: J102.1 (Pin_1), J102.2 (Pin_2) (x2)
- new net: J102.3 (Pin_3), J102.4 (Pin_4) (x2)
- new net: J243.1 (Pin_1), J243.2 (Pin_2)
- new net: J106.1 (Pin_1), J106.2 (Pin_2) (x2)
- new net: J106.3 (Pin_3), J106.4 (Pin_4) (x2)
- new net: J158.1 (Pin_1), J158.2 (Pin_2)
- new net: J238.1 (Pin_1), J238.2 (Pin_2)
- new net: J246.1 (Pin_1), J246.2 (Pin_2)
- new net: J242.1 (Pin_1), J242.2 (Pin_2)
- new net: J112.1 (Pin_1), J112.2 (Pin_2)
- new net: J112.3 (Pin_3), J112.4 (Pin_4)
- new net: J120.1 (Pin_1), J120.2 (Pin_2) (x2)
- new net: J120.3 (Pin_3), J120.4 (Pin_4)
- new net: J247.1 (Pin_1), J247.2 (Pin_2)
- new net: J232.1 (Pin_1), J232.2 (Pin_2), J232.3 (Pin_3)
- new net: J230.1 (Pin_1), J230.2 (Pin_2)
- new net: J123.1 (Pin_1), J123.2 (Pin_2) (x2)
- new net: J244.1 (Pin_1), J244.2 (Pin_2)
- new net: J100.1 (Pin_1), J100.2 (Pin_2)
- new net: J100.3 (Pin_3), J100.4 (Pin_4)
- new net: J236.1 (Pin_1), J236.2 (Pin_2)
- new net: J236.3 (Pin_3), J236.4 (Pin_4)
- new net: J182.1 (Pin_1), J182.2 (Pin_2)
- new net: J111.1 (Pin_1), J111.2 (Pin_2) (x2)
- new net: J111.3 (Pin_3), J111.4 (Pin_4) (x2)
- new net: J137.1 (Pin_1), J137.2 (Pin_2), J137.3 (Pin_3)
- new net: J130.1 (Pin_1), J130.2 (Pin_2)
- new net: J130.3 (Pin_3), J130.4 (Pin_4)
- new net: J237.1 (Pin_1), J237.2 (Pin_2)
- new net: J237.3 (Pin_3), J237.4 (Pin_4)
- new net: J123.3 (Pin_3), J123.4 (Pin_4)
- new net: J181.1 (Pin_1), J181.2 (Pin_2), J181.3 (Pin_3), J181.4 (Pin_4), J181.5 (Pin_5)
- new net: J178.1 (Pin_1), J178.2 (Pin_2)
- new net: J178.3 (Pin_3), J178.4 (Pin_4)
- new net: J108.1 (Pin_1), J108.2 (Pin_2) (x2)
- new net: J128.1 (Pin_1), J128.2 (Pin_2)
- new net: J128.3 (Pin_3), J128.4 (Pin_4)
- new net: J116.1 (Pin_1), J116.2 (Pin_2) (x2)
- new net: J116.3 (Pin_3), J116.4 (Pin_4) (x2)
- new net: J99.1 (Pin_1), J99.2 (Pin_2) (x2)
- new net: J99.3 (Pin_3), J99.4 (Pin_4) (x2)
- new net: J132.1 (Pin_1), J132.2 (Pin_2), J132.3 (Pin_3)
- new net: J240.1 (Pin_1), J240.2 (Pin_2)
- new net: J240.3 (Pin_3), J240.4 (Pin_4)
- new net: J165.1 (Pin_1), J165.2 (Pin_2)
- new net: J119.1 (Pin_1), J119.2 (Pin_2) (x2)
- new net: J113.1 (Pin_1), J113.2 (Pin_2) (x2)
- new net: J113.3 (Pin_3), J113.4 (Pin_4)
- new net: J98.1 (Pin_1), J98.2 (Pin_2) (x2)
- new net: J98.3 (Pin_3), J98.4 (Pin_4) (x2)
- new net: J98.5 (Pin_5), J98.6 (Pin_6)
- new net: J98.7 (Pin_7), J98.8 (Pin_8)
- new net: J161.1 (Pin_1), J161.2 (Pin_2)
- new net: J161.3 (Pin_3), J161.4 (Pin_4)
- new net: J164.1 (Pin_1), J164.2 (Pin_2)
- new net: J163.1 (Pin_1), J163.2 (Pin_2)
- new net: J163.3 (Pin_3), J163.4 (Pin_4)
- new net: J97.1 (Pin_1), J97.2 (Pin_2) (x2)
- new net: J97.3 (Pin_3), J97.4 (Pin_4) (x2)
- new net: J168.1 (Pin_1), J168.2 (Pin_2), J168.3 (Pin_3), J168.4 (Pin_4)
- new net: J101.1 (Pin_1), J101.2 (Pin_2) (x2)
- new net: J101.3 (Pin_3), J101.4 (Pin_4)
- new net: J114.1 (Pin_1), J114.2 (Pin_2) (x2)
- new net: J114.3 (Pin_3), J114.4 (Pin_4)
- new net: J105.1 (Pin_1), J105.2 (Pin_2) (x2)
- new net: J105.3 (Pin_3), J105.4 (Pin_4) (x2)
- new net: J104.1 (Pin_1), J104.2 (Pin_2) (x2)
- new net: J104.3 (Pin_3), J104.4 (Pin_4)
- new net: J90.1 (Pin_1), J90.2 (Pin_2) (x2)
- new net: J129.1 (Pin_1), J129.2 (Pin_2)
- new net: J129.3 (Pin_3), J129.4 (Pin_4)
- new net: J138.1 (Pin_1), J138.2 (Pin_2)
- new net: J138.3 (Pin_3), J138.4 (Pin_4)
- new net: J117.1 (Pin_1), J117.2 (Pin_2)
- new net: J117.3 (Pin_3), J117.4 (Pin_4)
- new net: J118.1 (Pin_1), J118.2 (Pin_2) (x2)
- new net: J227.1 (Pin_1), J227.2 (Pin_2)
- new net: J227.3 (Pin_3), J227.4 (Pin_4)
- new net: J133.1 (Pin_1), J133.2 (Pin_2), J133.3 (Pin_3), J133.4 (Pin_4)
- new net: J122.1 (Pin_1), J122.2 (Pin_2) (x2)
- new net: J90.3 (Pin_3), J90.4 (Pin_4)
- new net: J170.1 (Pin_1), J170.2 (Pin_2)
- new net: J107.1 (Pin_1), J107.2 (Pin_2) (x2)
- new net: J107.3 (Pin_3), J107.4 (Pin_4)
- new net: J180.1 (Pin_1), J180.2 (Pin_2)
- new net: J180.3 (Pin_3), J180.4 (Pin_4)
- new net: J228.1 (Pin_1), J228.2 (Pin_2)
- new net: J228.3 (Pin_3), J228.4 (Pin_4)
- new net: J177.1 (Pin_1), J177.2 (Pin_2), J177.3 (Pin_3), J177.4 (Pin_4), J177.5 (Pin_5)
- new net: J122.3 (Pin_3), J122.4 (Pin_4)
- new net: J135.1 (Pin_1), J135.2 (Pin_2), J135.3 (Pin_3), J135.4 (Pin_4)
- new net: J234.1 (Pin_1), J234.2 (Pin_2)
- new net: J234.3 (Pin_3), J234.4 (Pin_4)
- new net: J235.1 (Pin_1), J235.2 (Pin_2)
- new net: J239.1 (Pin_1), J239.2 (Pin_2)
- new net: J239.3 (Pin_3), J239.4 (Pin_4)
- new net: J159.1 (Pin_1), J159.2 (Pin_2)
- new net: J159.3 (Pin_3), J159.4 (Pin_4)
- new net: J245.1 (Pin_1), J245.2 (Pin_2)
- new net: J173.1 (Pin_1), J173.2 (Pin_2)
- new net: J109.1 (Pin_1), J109.2 (Pin_2) (x2)
- new net: J109.3 (Pin_3), J109.4 (Pin_4)
- new net: J117.1 (Pin_1), J117.2 (Pin_2), J117.3 (Pin_3), J117.4 (Pin_4), J117.5 (Pin_5)
- new net: J108.3 (Pin_3), J108.4 (Pin_4)
- new net: J241.1 (Pin_1), J241.2 (Pin_2), J241.3 (Pin_3)
- new net: J233.1 (Pin_1), J233.2 (Pin_2)
- new net: J233.3 (Pin_3), J233.4 (Pin_4)
- new net: J179.1 (Pin_1), J179.2 (Pin_2), J179.3 (Pin_3), J179.4 (Pin_4)
- new net: J115.1 (Pin_1), J115.2 (Pin_2) (x2)
- new net: J115.3 (Pin_3), J115.4 (Pin_4)
- new net: J110.1 (Pin_1), J110.2 (Pin_2) (x2)
- new net: J110.3 (Pin_3), J110.4 (Pin_4) (x2)
- new net: J127.1 (Pin_1), J127.2 (Pin_2)
- new net: J127.3 (Pin_3), J127.4 (Pin_4)
- new net: J119.3 (Pin_3), J119.4 (Pin_4)
- new net: J121.1 (Pin_1), J121.2 (Pin_2)
- new net: J118.3 (Pin_3), J118.4 (Pin_4)
- new net: J126.1 (Pin_1), J126.2 (Pin_2)
- new net: J126.3 (Pin_3), J126.4 (Pin_4)
- new net: J174.1 (Pin_1), J174.2 (Pin_2)
- new net: J136.1 (Pin_1), J136.2 (Pin_2), J136.3 (Pin_3), J136.4 (Pin_4), J136.5 (Pin_5)
- new net: J217.1 (Pin_1), J217.2 (Pin_2)
- new net: J160.1 (Pin_1), J160.2 (Pin_2)
- new net: J160.3 (Pin_3), J160.4 (Pin_4)
- new net: J157.1 (Pin_1), J157.2 (Pin_2)
- new net: J157.3 (Pin_3), J157.4 (Pin_4)
- new net: J103.1 (Pin_1), J103.2 (Pin_2)
- new net: J103.3 (Pin_3), J103.4 (Pin_4)
- new net: J124.1 (Pin_1), J124.2 (Pin_2)
- new net: J124.3 (Pin_3), J124.4 (Pin_4)
- new net: J229.1 (Pin_1), J229.2 (Pin_2)
- new net: J229.3 (Pin_3), J229.4 (Pin_4)
- new net: J131.1 (Pin_1), J131.2 (Pin_2)
- new net: J131.3 (Pin_3), J131.4 (Pin_4)
- new net: J248.1 (Pin_1), J248.2 (Pin_2)
- new net: J231.1 (Pin_1), J231.2 (Pin_2)
- new net: J231.3 (Pin_3), J231.4 (Pin_4)
Other:
- note added: "<300mm STUBS NO LONGER IF THERE ARE ISSUES I AM CUTTING THEM OFF"
- note added: "AIRBRIDGE"
- note added: "BACK"
- note added: "BMS"
- note added: "CAN AIRBRIDGE - filtered bus to not overload bridge"
- note added: "CAN ISOLATED - electically isolated bus from TEMs"
- note added: "CAN REPEATER"
- note added: "CAN SENSOR - has sensor devices. is not needed to run car"
- note added: "CAN TRACTIVE - has all devices related to TS"
- note added: "Crimp x2 CAN H and x2 CAN L into connector"
- note added: "DASH"
- note added: "DASH BOX"
- note added: "FIREWALL"
- note added: "FRONT"
- note added: "FWPS"
- note added: "GPS"
- note added: "IN AND OUT Crimp x2 H and x2 L into connector"
- note added: "IN AND OUT Crimp x2 HL into connector"
- note added: "INVERTER"
- note added: "INVERTER RS232 - for programming the inverter"
- note added: "ISOCAN REPEATER"
- note added: "KVASER USB - for offloading memrata data"
- note added: "LABLES"
- note added: "LSPS"
- note added: "LV BOX"
- note added: "MEMORATOR"
- note added: "MEMORATOR PRO"
- note added: "MOTEC ETHERNET - for offloading L120 data"
- note added: "MOTEC L120"
- note added: "MOTEC PDM"
- note added: "PCB passthrough"
- note added: "PEDAL BOX"
- note added: "PITOT"
- note added: "REAR BOX"
- note added: "RSPS"
- note added: "RWPS"
- note added: "SENSOR HUB"
- note added: "TEMS"
- note added: "TSAC"
- note added: "UMBILICAL"
- note added: "VCU"
- note added: "blanking cap needed"
- note added: "filter messages for airbridge"
- note added: "if fwps not run, could terminate here"
- note added: "order in box not fixed"
- note added: "repeat all messages from I to T"
- note added: "splice MUST be inside backshell to be protected. make as close to connector as possible"
- note added: "terminate"
- note added: "terminate on PCB"
