File: Stag12/CAN.kicad_sch (KiCad schematic)
At the start: 68 parts, among them J100 Conn_02x02_Counter_Clockwise, J101 Conn_02x02_Counter_Clockwise, J102 Conn_02x02_Counter_Clockwise, J105 Conn_02x02_Counter_Clockwise, J106 Conn_02x02_Counter_Clockwise, J107 Conn_02x02_Counter_Clockwise, J108 Conn_01x02, J109 Conn_01x02, J110 Conn_02x02_Counter_Clockwise, J111 Conn_02x02_Counter_Clockwise, J113 Conn_02x02_Counter_Clockwise, J114 Conn_02x02_Counter_Clockwise, J115 Conn_01x02, J116 Conn_02x02_Counter_Clockwise, J117 Conn_02x02_Counter_Clockwise, J118 Conn_02x02_Counter_Clockwise, J119 Conn_02x02_Counter_Clockwise, J120 Conn_02x02_Counter_Clockwise, J121 Conn_02x02_Counter_Clockwise, J122 Conn_02x02_Counter_Clockwise, J123 Conn_02x02_Counter_Clockwise, J124 Conn_02x02_Counter_Clockwise, J126 Conn_02x02_Counter_Clockwise, J127 Conn_02x02_Counter_Clockwise, J128 Conn_02x02_Counter_Clockwise, J129 Conn_02x02_Counter_Clockwise, J130 Conn_02x02_Counter_Clockwise, J131 Conn_02x02_Counter_Clockwise, J132 Conn_01x03, J133 Conn_01x04, J134 Conn_01x05, J135 Conn_01x04, J136 Conn_01x05, J137 Conn_01x03, J138 Conn_02x02_Counter_Clockwise, J67 Conn_02x02_Counter_Clockwise, J68 Conn_02x02_Counter_Clockwise, J69 Conn_02x02_Counter_Clockwise, J70 Conn_01x02, J71 Conn_02x02_Counter_Clockwise, J72 Conn_01x02, J73 Conn_01x02, J74 Conn_01x02, J75 Conn_01x02, J76 Conn_01x02, J77 Conn_01x02, J78 Conn_01x02, J79 Conn_01x02, J80 Conn_02x02_Counter_Clockwise, J81 Conn_02x02_Counter_Clockwise, J82 Conn_02x02_Counter_Clockwise, J83 Conn_02x02_Counter_Clockwise, J84 Conn_02x02_Counter_Clockwise, J85 Conn_02x02_Counter_Clockwise, J86 Conn_02x02_Counter_Clockwise, J87 Conn_02x02_Counter_Clockwise, J88 Conn_02x02_Counter_Clockwise, J89 Conn_02x02_Counter_Clockwise, J90 Conn_02x02_Counter_Clockwise, J91 Conn_02x02_Counter_Clockwise, J92 Conn_02x02_Counter_Clockwise, J93 Conn_02x02_Counter_Clockwise, J94 Conn_02x02_Counter_Clockwise, J95 Conn_02x02_Counter_Clockwise, J96 Conn_02x02_Counter_Clockwise, J97 Conn_02x02_Counter_Clockwise, J98 Conn_02x04_Counter_Clockwise, J99 Conn_02x02_Counter_Clockwise

Commit message: Updated can
Parts:
- removed J100, J101, J68, J80, J82, J83: Conn_02x02_Counter_Clockwise, symbol Connector_Generic:Conn_02x02_Counter_Clockwise
- removed J134: Conn_01x05, symbol Connector_Generic:Conn_01x05
- removed J74: Conn_01x02, symbol Connector_Generic:Conn_01x02
- added J101, J104, J158, J164, J165, J170, J173, J174, J182, J217, J230, J235, J238, J242, J243, J244, J245, J246, J248, J80, J83: Conn_01x02, symbol Connector_Generic:Conn_01x02
- added J157, J159, J160, J161, J163, J169, J178, J180, J227, J228, J229, J231, J233, J234, J236, J237, J239, J240, J247, J74: Conn_02x02_Counter_Clockwise, symbol Connector_Generic:Conn_02x02_Counter_Clockwise
- added J168, J179: Conn_01x04, symbol Connector_Generic:Conn_01x04
- added J177, J181, J68: Conn_01x05, symbol Connector_Generic:Conn_01x05
- added J232, J241: Conn_01x03, symbol Connector_Generic:Conn_01x03
Connections:
- net at J121.1 (Pin_1): no longer J121.2 (Pin_2)
- net at J121.3 (Pin_3): no longer J121.4 (Pin_4)
- new net: J169.1 (Pin_1), J169.2 (Pin_2)
- new net: J169.3 (Pin_3), J169.4 (Pin_4)
- new net: J243.1 (Pin_1), J243.2 (Pin_2)
- new net: J158.1 (Pin_1), J158.2 (Pin_2)
- new net: J238.1 (Pin_1), J238.2 (Pin_2)
- new net: J246.1 (Pin_1), J246.2 (Pin_2)
- new net: J242.1 (Pin_1), J242.2 (Pin_2)
- new net: J247.1 (Pin_1), J247.2 (Pin_2)
- new net: J232.1 (Pin_1), J232.2 (Pin_2), J232.3 (Pin_3)
- new net: J230.1 (Pin_1), J230.2 (Pin_2)
- new net: J244.1 (Pin_1), J244.2 (Pin_2)
- new net: J236.1 (Pin_1), J236.2 (Pin_2)
- new net: J236.3 (Pin_3), J236.4 (Pin_4)
- new net: J182.1 (Pin_1), J182.2 (Pin_2)
- new net: J237.1 (Pin_1), J237.2 (Pin_2)
- new net: J237.3 (Pin_3), J237.4 (Pin_4)
- new net: J181.1 (Pin_1), J181.2 (Pin_2), J181.3 (Pin_3), J181.4 (Pin_4), J181.5 (Pin_5)
- new net: J178.1 (Pin_1), J178.2 (Pin_2)
- new net: J178.3 (Pin_3), J178.4 (Pin_4)
- new net: J240.1 (Pin_1), J240.2 (Pin_2)
- new net: J240.3 (Pin_3), J240.4 (Pin_4)
- new net: J165.1 (Pin_1), J165.2 (Pin_2)
- new net: J68.1 (Pin_1), J68.2 (Pin_2), J68.3 (Pin_3), J68.4 (Pin_4), J68.5 (Pin_5)
- new net: J161.1 (Pin_1), J161.2 (Pin_2)
- new net: J161.3 (Pin_3), J161.4 (Pin_4)
- new net: J164.1 (Pin_1), J164.2 (Pin_2)
- new net: J163.1 (Pin_1), J163.2 (Pin_2)
- new net: J163.3 (Pin_3), J163.4 (Pin_4)
- new net: J168.1 (Pin_1), J168.2 (Pin_2), J168.3 (Pin_3), J168.4 (Pin_4)
- new net: J80.1 (Pin_1), J80.2 (Pin_2)
- new net: J227.1 (Pin_1), J227.2 (Pin_2)
- new net: J227.3 (Pin_3), J227.4 (Pin_4)
- new net: J170.1 (Pin_1), J170.2 (Pin_2)
- new net: J180.1 (Pin_1), J180.2 (Pin_2)
- new net: J180.3 (Pin_3), J180.4 (Pin_4)
- new net: J228.1 (Pin_1), J228.2 (Pin_2)
- new net: J228.3 (Pin_3), J228.4 (Pin_4)
- new net: J177.1 (Pin_1), J177.2 (Pin_2), J177.3 (Pin_3), J177.4 (Pin_4), J177.5 (Pin_5)
- new net: J74.1 (Pin_1), J74.2 (Pin_2)
- new net: J74.3 (Pin_3), J74.4 (Pin_4)
- new net: J234.1 (Pin_1), J234.2 (Pin_2)
- new net: J234.3 (Pin_3), J234.4 (Pin_4)
- new net: J235.1 (Pin_1), J235.2 (Pin_2)
- new net: J239.1 (Pin_1), J239.2 (Pin_2)
- new net: J239.3 (Pin_3), J239.4 (Pin_4)
- new net: J159.1 (Pin_1), J159.2 (Pin_2)
- new net: J159.3 (Pin_3), J159.4 (Pin_4)
- new net: J245.1 (Pin_1), J245.2 (Pin_2)
- new net: J173.1 (Pin_1), J173.2 (Pin_2)
- new net: J241.1 (Pin_1), J241.2 (Pin_2), J241.3 (Pin_3)
- new net: J233.1 (Pin_1), J233.2 (Pin_2)
- new net: J233.3 (Pin_3), J233.4 (Pin_4)
- new net: J179.1 (Pin_1), J179.2 (Pin_2), J179.3 (Pin_3), J179.4 (Pin_4)
- new net: J174.1 (Pin_1), J174.2 (Pin_2)
- new net: J217.1 (Pin_1), J217.2 (Pin_2)
- new net: J160.1 (Pin_1), J160.2 (Pin_2)
- new net: J160.3 (Pin_3), J160.4 (Pin_4)
- new net: J104.1 (Pin_1), J104.2 (Pin_2)
- new net: J157.1 (Pin_1), J157.2 (Pin_2)
- new net: J157.3 (Pin_3), J157.4 (Pin_4)
- new net: J101.1 (Pin_1), J101.2 (Pin_2)
- new net: J229.1 (Pin_1), J229.2 (Pin_2)
- new net: J229.3 (Pin_3), J229.4 (Pin_4)
- new net: J248.1 (Pin_1), J248.2 (Pin_2)
- new net: J83.1 (Pin_1), J83.2 (Pin_2)
- new net: J231.1 (Pin_1), J231.2 (Pin_2)
- new net: J231.3 (Pin_3), J231.4 (Pin_4)
Other:
- note added: "<300mm STUBS NO LONGER IF THERE ARE ISSUES I AM CUTTING THEM OFF"
- note added: "Crimp x2 CAN H and x2 CAN L into connector"
- note added: "IN AND OUT Crimp x2 H and x2 L into connector"
- note added: "IN AND OUT Crimp x2 HL into connector"
- note added: "MEMORATOR PRO"
- note added: "PCB passthrough"
- note added: "terminate on PCB"
- note removed: "repeat select messages from T to S"
- note removed: "spur as close to pdm as possible"
- note removed: "work out wtf to do here, thinking in and out to a dtm but needs then blanking cap"
- moved on the sheet: J106, J107, J108, J109, J110, J111, J113, J114, J116, J117, J118, J119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

Commit message: CAN changes
Parts:
- removed J102, J106, J107, J110, J111, J113, J114, J116, J117, J118, J119, J120, J121, J123, J126, J127, J128, J129, J130, J131, J163, J227, J228, J247, J74: Conn_02x02_Counter_Clockwise, symbol Connector_Generic:Conn_02x02_Counter_Clockwise
- removed J104, J108, J109, J115, J244, J245, J246, J248, J73, J75, J76, J77, J78, J79, J80: Conn_01x02, symbol Connector_Generic:Conn_01x02
- removed J132, J137: Conn_01x03, symbol Connector_Generic:Conn_01x03
- removed J133, J135: Conn_01x04, symbol Connector_Generic:Conn_01x04
- removed J136, J68: Conn_01x05, symbol Connector_Generic:Conn_01x05
- added J68: Conn_02x02_Counter_Clockwise, symbol Connector_Generic:Conn_02x02_Counter_Clockwise
Connections:
- net at J71.3 (Pin_3): no longer J71.4 (Pin_4)
- new net: J68.1 (Pin_1), J68.2 (Pin_2)
Other:
- note added: "CAN Isolator"
- note added: "Terminate"
- note removed: "IN AND OUT Crimp x2 HL into connector"
- note removed: "ISOCAN REPEATER"
- note removed: "MEMORATOR PRO"
- moved on the sheet: J101, J105, J122, J138, J157, J158, J159, J160, J161, J164, J165, J168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
