File: Stag12/device/device-tsal.kicad_sch (KiCad schematic)
At the start: 9 parts

Commit message: Changed EXCs to PWRs
any mention of exc switched to pwr :)
Changed lines of the file:
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@@
 		)
 	)
-	(label "TSAL.LED.EXC"
+	(label "TSAL.LED.PWR"
 		(at 73.66 57.15 0)
 		(effects
