File: Stag12/loom/LOOM - HV BOX.kicad_sch (KiCad schematic)
At the start: 16 parts, among them SW12 Hirose EM30MSD

Commit message: Changed EXCs to PWRs
any mention of exc switched to pwr :)
Connections:
- net BSPD.CUR_SEN.EXC renamed BSPD.CUR_SEN.PWR
- net HVSENSE.EXC renamed HVSENSE.PWR
Changed lines of the file:
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@@
 		)
 	)
-	(label "BSPD.CUR_SEN.EXC"
+	(label "BSPD.CUR_SEN.PWR"
 		(at 39.37 26.67 0)
 		(effects
@@
 		)
 	)
-	(label "REB.HVS.EXC"
+	(label "REB.HVS.PWR"
 		(at 242.57 140.335 180)
 		(effects
@@
 		)
 	)
-	(label "BSPD.CUR_SEN.EXC"
+	(label "BSPD.CUR_SEN.PWR"
 		(at 57.15 161.29 180)
 		(effects
@@
 		)
 	)
-	(label "HVSENSE.EXC"
+	(label "HVSENSE.PWR"
 		(at 39.37 21.59 0)
 		(effects
