File: Stag12/loom/LOOM - HV BOX.kicad_sch (KiCad schematic)
At the start: 16 parts, among them SW12 Hirose EM30MSD

Commit message: Whole bunch of mid-build fixes and notes i think
Parts:
- added J195: Conn_01x12_Socket, symbol Connector:Conn_01x12_Socket
- added J196: Conn_01x04_Socket, symbol Connector:Conn_01x04_Socket
Connections:
- no-connect marks 6 -> 9
Other:
- note added: "USING THIS PINOUT!"

Commit message: commit changes from before comp
Other:
- note added: "gnd"
- note added: "pwr"
- note added: "sig"
Changed lines of the file:
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@@
+		)
+	)
+	(text "gnd"
+		(exclude_from_sim no)
+		(at 61.722 100.33 0)
+		(effects
+			(font
+				(size 1.27 1.27)
+			)
 		)
 	)
@@
 		)
 	)
+	(text "pwr"
+		(exclude_from_sim no)
+		(at 61.976 102.87 0)
+		(effects
+			(font
+				(size 1.27 1.27)
+			)
+		)
+	)
 	(text "USING THIS PINOUT!"
 		(exclude_from_sim no)
@@
 			)
 		)
+	)
+	(text "sig"
+		(exclude_from_sim no)
+		(at 61.722 97.79 0)
+		(effects
+			(font
+				(size 1.27 1.27)
+			)
+		)
