File: Stag12/loom/loom-umbilical-box.kicad_sch (KiCad schematic)
At the start: 0 parts

Commit message: idfk
Parts:
- added D7: PWR LED, symbol Device:LED
- added SW13: LV Enable, symbol Switch:SW_SPST
- added SW15: LV Reset, symbol Switch:SW_Push
- added SW16: GLV Bypass, symbol Switch:SW_Push
- added SW17: E-STOP, symbol Switch:SW_Push
- added SW18: Power Routing, symbol Switch:SW_SPST
Connections:
- new net E-STOP: SW17.1
- new net GLV.BYP ?????: SW16.1
- new net GND: SW15.2, SW16.2, SW17.2
- new net LV.EN +: SW13.1 (A)
- new net LV.EN -: SW13.2 (B)
- new net LV.RST: SW15.1
- new net PWR +: D7.2 (A), SW18.1 (A)
- new net PWR -: D7.1 (K), SW18.2 (B)
