File: Stag12/loom/LOOM - LV BOX.kicad_sch (KiCad schematic)
At the start: 27 parts, among them J10 LATCHING, J8 TSAL, J9 POWER

Commit message: Changed EXCs to PWRs
any mention of exc switched to pwr :)
Connections:
- net CAN.NODE.EXC renamed CAN.NODE.PWR
- net REB.HVS.EXC renamed REB.HVS.PWR
- net RTDS.EXC renamed RTDS.PWR
- net TSAL_LATCHING.EXC renamed TSAL_LATCHING.PWR
- net VCU.EXC renamed VCU.PWR
Changed lines of the file:
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@@
 		)
 	)
-	(label "TSAL.DASH.EXC"
+	(label "TSAL.DASH.PWR"
 		(at 529.59 241.3 180)
 		(effects
@@
 		)
 	)
-	(label "IMD.LED.EXC"
+	(label "IMD.LED.PWR"
 		(at 527.05 180.34 180)
 		(effects
@@
 		)
 	)
-	(label "PWR_SPLICE.EXC"
+	(label "PWR_SPLICE.PWR"
 		(at 57.15 40.64 0)
 		(effects
@@
 		)
 	)
-	(label "REB.HVS.EXC"
+	(label "REB.HVS.PWR"
 		(at 57.15 179.07 0)
 		(effects
@@
 		)
 	)
-	(label "LATCHING.EXC"
+	(label "LATCHING.PWR"
 		(at 162.56 17.78 0)
 		(effects
@@
 		)
 	)
-	(label "TSAL.DASH.EXC"
+	(label "TSAL.DASH.PWR"
 		(at 57.15 45.72 0)
 		(effects
@@
 		)
 	)
-	(label "RTDS.EXC"
+	(label "RTDS.PWR"
 		(at 525.78 91.44 180)
 		(effects
@@
 		)
 	)
-	(label "BMS.LED.EXC"
+	(label "BMS.LED.PWR"
 		(at 527.05 177.8 180)
 		(effects
@@
 		)
 	)
-	(label "TSAL.LED.EXC"
+	(label "TSAL.LED.PWR"
 		(at 529.59 233.68 180)
 		(effects
@@
 		)
 	)
-	(label "CAN.NODE.EXC"
+	(label "CAN.NODE.PWR"
 		(at 58.42 283.21 0)
 		(effects
@@
 		)
 	)
-	(label "REB.HVS.EXC"
+	(label "REB.HVS.PWR"
 		(at 529.59 238.76 180)
 		(effects
@@
 		)
 	)
-	(label "SPARE.EXC"
+	(label "SPARE.PWR"
 		(at 525.78 76.2 180)
 		(effects
@@
 		)
 	)
-	(label "TS.ON.LED.EXC"
+	(label "TS.ON.LED.PWR"
 		(at 527.05 172.72 180)
 		(effects
@@
 		)
 	)
-	(label "TSAL.EXC"
+	(label "TSAL.PWR"
 		(at 162.56 27.94 0)
 		(effects
@@
 		)
 	)
-	(label "TSAC.HVS.EXC"
+	(label "TSAC.HVS.PWR"
 		(at 529.59 236.22 180)
 		(effects
@@
 		)
 	)
-	(label "TS.ON.BUTTON.EXC"
+	(label "TS.ON.BUTTON.PWR"
 		(at 527.05 170.18 180)
 		(effects
@@
 		)
 	)
-	(label "TSAC.HVS.EXC"
+	(label "TSAC.HVS.PWR"
 		(at 57.15 104.14 0)
 		(effects
@@
 		)
 	)
-	(label "TSAL.LED.EXC"
+	(label "TSAL.LED.PWR"
 		(at 57.15 58.42 0)
 		(effects
@@
 		)
 	)
-	(label "R2D.LED.EXC"
+	(label "R2D.LED.PWR"
 		(at 527.05 175.26 180)
 		(effects
@@
 		)
 	)
-	(label "TSAL_LATCHING.EXC"
+	(label "TSAL_LATCHING.PWR"
 		(at 529.59 246.38 180)
 		(effects
@@
 		)
 	)
-	(label "RTDS.EXC"
+	(label "RTDS.PWR"
 		(at 57.15 83.82 0)
 		(effects
@@
 		)
 	)
-	(label "PWR_SPLICE.EXC"
+	(label "PWR_SPLICE.PWR"
 		(at 58.42 269.24 0)
 		(effects
@@
 		)
 	)
-	(label "VCU.EXC"
+	(label "VCU.PWR"
 		(at 527.05 121.92 180)
 		(effects
@@
 		)
 	)
-	(label "VCU.EXC"
+	(label "VCU.PWR"
 		(at 527.05 127 180)
 		(effects
@@
 		)
 	)
-	(label "VCU.EXC"
+	(label "VCU.PWR"
 		(at 162.56 22.86 0)
 		(effects
@@
 		)
 	)
-	(label "R2D.BUTTON.EXC"
+	(label "R2D.BUTTON.PWR"
 		(at 527.05 167.64 180)
 		(effects

Commit message: idfk
Other:
- note added: "fix me"
- note added: "tsac conected to tsal"
Changed lines of the file:
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@@
+		)
+	)
+	(text "tsac conected to tsal\n"
+		(exclude_from_sim no)
+		(at 38.862 107.696 0)
+		(effects
+			(font
+				(size 1.27 1.27)
+			)
 		)
 	)
@@
 		)
 	)
+	(text "fix me\n"
+		(exclude_from_sim no)
+		(at 40.64 110.49 0)
+		(effects
+			(font
+				(size 1.27 1.27)
+			)
+		)
+	)

Commit message: LV Box Redesign
Parts:
- removed Conn42, Conn44: Molex_4x2S_Recepticle, symbol Connectors_SUFST:Molex_4x2S_Recepticle
- removed Conn43: Molex_2x1S_Recepticle, symbol Connectors_SUFST:Molex_2x1S_Recepticle
- removed Conn45, Conn46, Conn47: Molex_2x2S_Recepticle, symbol Connectors_SUFST:Molex_2x2S_Recepticle
- removed Conn48: Molex_5x2S_Recepticle, symbol Connectors_SUFST:Molex_5x2S_Recepticle
- removed Conn49: Molex_3x2S_Recepticle, symbol Connectors_SUFST:Molex_3x2S_Recepticle
- removed Conn62: Deutsch_DTM_12S_Pin, symbol Connectors_SUFST:Deutsch_DTM_6S_Pin
- removed Conn88: TODO: CHECK CONNECTOR, symbol Connectors_SUFST:Deutsch_DTM_6P_Pin
- added Conn42: AMPHENOL-21P-Pannel, symbol Connectors_SUFST:AMPHENOL-21P-Pannel
- added Conn43: Conn A PDM Connector, symbol Connectors_SUFST:Conn A PDM Connector
- added Conn44: Conn C PDM Connector, symbol Connectors_SUFST:Conn C PDM Connector
- added J39: ASHD114-1SN-S25, symbol Connector_Generic:Conn_01x01
- Conn61: P/N AHDP06-24-47SR-SRA -> AHDP04-24-47SR-SRA
Connections:
- net APPS2.SIG is gone; now on net TSAL.RESET-: Conn61.2
- net BMS.FAULT.LATCHING is gone; now on net BMS.LED.K: J10.2 (Pin_2)
- net BPS.SIG is gone; now on net PDM.GND: Conn61.7
- net IMD.FAULT.LATCHING is gone; now on net IMD.LED.K: J10.1 (Pin_1)
- net RTDS.GND is gone; now on net LATCHING.RESET+: Conn61.22
- net RTDS.PWR is gone; now on net ~{BMS.FAULT}: Conn61.21
- net VCU.UART.RX is gone; now on net IMD.LED.K: Conn61.24
- net VCU.UART.TX is gone; now on net LATCHING.RESET-: Conn61.23
- net BATT+: no longer Conn61.46
- net BATT-: no longer Conn61.47
- net BMS.LED.K: now also Conn61.25; no longer Conn61.39
- net CAN.C.HIGH: now also Conn43.10; no longer Conn61.19
- net CAN.C.LOW: now also Conn43.9; no longer Conn61.20
- net CAN.NODE.GND: no longer Conn61.5
- net CAN.NODE.PWR: no longer Conn61.4
- net CAN.S.HIGH: no longer Conn61.25, Conn61.27
- net CAN.S.LOW: no longer Conn61.26, Conn61.28
- net IMD.LED.K: no longer Conn61.40
- net IMD.OK: now also Conn61.20; no longer Conn61.45
- net LATCHING.RESET+: no longer Conn61.41
- net LATCHING.RESET-: no longer Conn61.42
- net TS.DETECTED: now also Conn61.15, Conn61.30; no longer Conn61.17, Conn83.2
- net TS.ON: no longer Conn61.16, Conn81.2
- net TS.READY: no longer Conn61.9, Conn80.2
- net TSAL.GREEN.DASH.LED.K: now also Conn61.13; no longer Conn61.10
- net TSAL.GREEN.LED.EN: now also Conn61.11; no longer Conn61.13
- net TSAL.GREEN.LIGHT: now also Conn61.16; no longer Conn61.15, Conn82.2
- net TSAL.LED.GND: now also Conn61.10, J8.2 (Pin_2); no longer Conn61.14, J9.7 (Pin_7)
- net TSAL.PWR: now also Conn44.1
- net TSAL.RED.DASH.LED.K: now also Conn61.14
- net TSAL.RESET+: now also Conn61.8; no longer Conn61.32
- net TSAL.RESET-: no longer Conn61.31
- net TSAL_LATCHING.GND: now also Conn61.34
- net VOLTAGE.SHUT.TSAC.INTERLOCK.SIG: no longer Conn61.18
- net ~{BMS.DISCHARGE.ENABLE}: now also Conn61.19; no longer Conn61.43
- net ~{BMS.FAULT}: no longer Conn61.44
- net TSAL.LED.PWR: now reaches J8.1 (Pin_1)
- net TSAL.LED.PWR: now also Conn61.9
- net APPS1.SIG renamed PDM.GND
- net PDM.GND: now also Conn43.25, Conn43.26
- net CANNODE.HVS.SIG renamed VOLTAGE.CURRENT.SENSE.SIG
- net DRS.BUTTON.GND: no longer names the net of Conn61.33
- net R2D.BUTTON.GND: no longer names the net of Conn61.35
- net R2D.LED.K: no longer names the net of Conn61.38
- net REB.HVS.GND: no longer names the net of J9.9 (Pin_9)
- removed net REB.HVS.PWR: Conn61.11, Conn61.29, Conn61.6, J9.1 (Pin_1), J9.2 (Pin_2), J9.3 (Pin_3), J9.4 (Pin_4), J9.5 (Pin_5)
- net SAGL.SIG: no longer names the net of Conn79.2
- net SAGL.SIG: no longer Conn61.8
- net SHUT.HVD.INTERLOCK renamed SDC.FRONT
- net SDC.FRONT: now also Conn61.6; no longer Conn61.34, Conn85.2
- net SHUT.LATCHING renamed SDC.LATCHING
- net SDC.LATCHING: no longer Conn86.2
- net TS.ON.BUTTON.GND: no longer names the net of Conn61.36
- net TSAC.HVS.GND renamed HVSENSE.GND
- net HVSENSE.GND: now also Conn61.27; no longer Conn61.30
- net TSAL_LATCHING.PWR renamed LV_BOX.PWR
- net LV_BOX.PWR: now also Conn43.1
- new net BRAKE.LIGHT.PWR: Conn44.3
- new net CAN.C.H: Conn61.44, Conn61.46
- new net CAN.C.L: Conn61.45, Conn61.47
- new net DASHBOX.PWR: Conn43.2, Conn61.31
- new net FAN.PWR: Conn44.2
- new net HVSENSE.PWR: Conn61.26, J9.2 (Pin_2)
- new net IN.1: Conn43.4
- new net IN.10: Conn43.22
- new net IN.11: Conn43.23
- new net IN.12: Conn43.24
- new net IN.2: Conn43.5
- new net IN.3: Conn43.6
- new net IN.4: Conn43.16
- new net IN.5: Conn43.17
- new net IN.6: Conn43.18
- new net IN.7: Conn43.19
- new net IN.8: Conn43.20
- new net IN.9: Conn43.21
- new net INV.PWR: Conn44.6
- new net PDM.BATT+: Conn61.4, Conn61.5, J39.1 (Pin_1)
- new net PDM.GNDREF: Conn43.7, Conn43.8
- new net PUMP1.PWR: Conn44.4
- new net PUMP2.PWR: Conn44.5
- new net TRC.PWR: Conn61.28, J9.3 (Pin_3)
- new net TSAC.AUX.GND: Conn61.18, J9.7 (Pin_7)
- new net TSAC.AUX.PWR: Conn61.17, J9.1 (Pin_1)
- new net TSAL.DASH.PWR: Conn61.29, J9.4 (Pin_4)
- new net VOLTAGE.SHUT.HVD.INTERLOCK.SIG: Conn85.2
- new net VOLTAGE.SHUT.LATCHING.SIG: Conn86.2
- new net VOLTAGE.TS.DETECTED.SIG: Conn83.2
- new net VOLTAGE.TS.ON.SIG: Conn81.2
- new net VOLTAGE.TS.READY.SIG: Conn80.2
- new net VOLTAGE.~{GREEN.LED.ON}.SIG: Conn82.2
- no-connect marks 26 -> 1
Other:
- note added: "Is splice needed?"
- note added: "NC Key"
- note added: "OUT 20.1"
- note added: "OUT 20.2"
- note added: "OUT 20.3"
- note added: "OUT 20.4"
- note added: "OUT 20.5"
- note added: "OUT 20.6"
- note added: "OUT 8.10"
- note added: "OUT 8.11"
- note added: "OUT 8.12"
- note added: "OUT 8.13"
- note added: "OUT 8.14"
- note added: "OUT 8.15"
- note added: "OUT 8.16"
- note added: "OUT 8.9"
- note added: "SPARE OUTPUT 20.7"
- note added: "SPARE OUTPUT 20.8"
- note removed: "-->"
- note removed: "<--"
- note removed: "Change to socket molex"
- note removed: "I think we needed a 47 pin?"
- note removed: "Splice to CAN node and VCU"
- note removed: "TODO: CHECK IF IMD AND BMS GO TO DASH OR VCU"
- note removed: "TODO: SPEC Connectors for programmer (5 pin)"
- note removed: "TSAL Power wired wrong. No TSAL power to PWR_SPLICE"
- note removed: "VCU"
- note removed: "fix me"
- note removed: "tsac conected to tsal"
- moved on the sheet: Conn61, J10, J8, J9

Commit message: EMI hell
Parts:
- removed Conn43: Conn A PDM Connector, symbol Connectors_SUFST:Conn A PDM Connector
- removed Conn44: Conn C PDM Connector, symbol Connectors_SUFST:Conn C PDM Connector
- removed J39: ASHD114-1SN-S25, symbol Connector_Generic:Conn_01x01
- Conn61: symbol Connectors_SUFST:AMPHENOL-47P-Recepticle -> Connectors_SUFST:AMPHENOL-47P-Pannel; P/N AHDP04-24-47SR-SRA -> AHDP04-24-47PR-SRA
Connections:
- net TSAL.GREEN.LIGHT: no longer Conn61.16, J8.11 (Pin_11)
- net L120.GND: now reaches Conn61.43
- net LV_BOX.PWR renamed TSAL_LATCHING.PWR
- new net TRC.TSAL.GRN: Conn61.16, J8.11 (Pin_11)
Other:
- note added: "<- UPSTREAM"
- note added: "UPSTREAM ->"
- note removed: "OUT 20.1"
- note removed: "OUT 20.2"
- note removed: "OUT 20.3"
- note removed: "OUT 20.4"
- note removed: "OUT 20.5"
- note removed: "OUT 20.6"
- note removed: "OUT 8.10"
- note removed: "OUT 8.11"
- note removed: "OUT 8.12"
- note removed: "OUT 8.13"
- note removed: "OUT 8.14"
- note removed: "OUT 8.15"
- note removed: "OUT 8.16"
- note removed: "OUT 8.9"
- note removed: "SPARE OUTPUT 20.7"
- note removed: "SPARE OUTPUT 20.8"
- note removed: "TODO: Dash excitations, needed or no? Dash soft reset Maybe combine some EXC signals, not sure"

Commit message: Just one more layout
Parts:
- added Conn105: L120 Connector, symbol Connectors_SUFST:L120 Connector
Connections:
- net CAN.C.HIGH: now also Conn105.19
- net CAN.C.LOW: now also Conn105.18
- net L120.GND: now also Conn105.34
- new net CAN.B.HIGH: Conn105.27
- new net CAN.B.LOW: Conn105.26
- new net L120.ANALOGUE.TEMP.1: Conn105.16
- new net L120.ANALOGUE.TEMP.2: Conn105.17
- new net L120.ANALOGUE.VOLT.1: Conn105.3
- new net L120.ANALOGUE.VOLT.2: Conn105.4
- new net L120.ANALOGUE.VOLT.3: Conn105.5
- new net L120.ANALOGUE.VOLT.4: Conn105.6
- new net L120.ANALOGUE.VOLT.5: Conn105.12
- new net L120.ANALOGUE.VOLT.6: Conn105.13
- new net L120.DIGITAL.1: Conn105.14
- new net L120.DIGITAL.2: Conn105.15
- new net L120.ERX+: Conn105.11
- new net L120.ERX-: Conn105.10
- new net L120.ETX+: Conn105.2
- new net L120.ETX-: Conn105.1
- new net L120.PWR: Conn105.33
- new net L120.SENSOR.5V: Conn105.8
- new net L120.SENSOR.8V: Conn105.7
- new net L120.SENSOR.GND: Conn105.9
- new net L120.SPEED.1: Conn105.21
- new net L120.SPEED.2: Conn105.22
- new net L120.SPEED.3: Conn105.23
- new net RS232-1 RX: Conn105.28
- new net RS232-1 TX: Conn105.20
- new net RS232-2 RX: Conn105.25
- no-connect marks 1 -> 23
Other:
- note added: "25mA MAXIMUM RECOMMENDED TO USE EXTERNAL POWER"
- note added: "CRIMP TO GND"
- note added: "TODO: CHECK 15V TOLERANT INPUT"
- note added: "|- | AUX output| |_"

Commit message: Top loom and LV box?
Parts:
- removed Conn75, Conn76, Conn77, Conn78, Conn79, Conn80, Conn81, Conn82, Conn83, Conn84, Conn85, Conn86: Molex_2x1S_Recepticle, symbol Connectors_SUFST:Molex_2x1S_Recepticle
- removed Conn87: Molex_4x1S_Recepticle, symbol Connectors_SUFST:Molex_4x1S_Recepticle
- added Conn2: AMPHENOL-47P-Recepticle, symbol Connectors_SUFST:AMPHENOL-47P-Pannel
- added J13: POWER, Connector_Molex:Molex_Micro-Fit_3.0_43045-1200_2x06_P3.00mm_Horizontal, symbol Connector_Generic:Conn_01x12
- added J14: LATCHING, Connector_Molex:Molex_Micro-Fit_3.0_43045-1200_2x06_P3.00mm_Horizontal, symbol Connector_Generic:Conn_01x12
- added J5: TSAL, Connector_Molex:Molex_Micro-Fit_3.0_43045-1200_2x06_P3.00mm_Horizontal, symbol Connector_Generic:Conn_01x12
- added J64, J66: Conn_01x12, symbol Connector_Generic:Conn_01x12
- added J68: Conn_01x12, symbol Connector_Generic:Conn_01x04
Connections:
- no-connect marks 23 -> 24
Other:
- note added: "8Ch Sensor Hub"
- note added: "BOTTOM LEFT"
- note added: "CAN REPEATER"
- note added: "GND +GLV CANH CANL"
- note added: "L1 GND 3V3"
- note added: "L2 GND 3V3"
- note added: "L3 GND 3V3"
- note added: "L4 GND 3V3"
- note added: "L5 GND 3V3"
- note added: "L6 GND 3V3"
- note added: "L7 GND 3V3"
- note added: "L8 GND 3V3"
- note added: "Molex 43045-1200"
- note added: "TOP LEFT"
- note removed: "CAN-NODE"
- note removed: "PWR and DATA"
- note removed: "Temperature 1"
- note removed: "Temperature 2"
- note removed: "Voltage 1"
- note removed: "Voltage 10"
- note removed: "Voltage 2"
- note removed: "Voltage 3"
- note removed: "Voltage 4"
- note removed: "Voltage 5"
- note removed: "Voltage 6"
- note removed: "Voltage 7"
- note removed: "Voltage 8"
- note removed: "Voltage 9"
- moved on the sheet: Conn105, Conn42, Conn61, J10, J8, J9
