File: Stag12/loom/loom-top.kicad_sch (KiCad schematic)
At the start: 3 parts

Commit message: Updated top loom connector
Parts:
- Conn60: symbol Connectors_SUFST:Deutsch_DTM_12S_Pin -> Connectors_SUFST:AT16-18SA; P/N AT/DT Plug, 12pos -> AT16-18SA
Other:
- note added: "Might be 09 9764 70 04 Warwick might know?"
Changed lines of the file:
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@@
 	(generator_version "9.0")
 	(paper "A4")
+	(text "Might be\n09 9764 70 04\n\nWarwick might know?"
+		(exclude_from_sim no)
+		(at 233.172 114.554 0)
+		(effects
+			(font
+				(size 1.27 1.27)
+			)
+		)
+	)
 	(wire
 		(pts
@@
 	)
 	(symbol
-		(lib_id "Connectors_SUFST:Deutsch_DTM_12S_Pin")
+		(lib_id "Connectors_SUFST:AT16-18SA")
 		(at 52.07 101.6 0)
 		(mirror x)
@@
 			)
 		)
-		(property "P/N" "AT/DT Plug, 12pos"
-			(at 38.735 83.185 0)
+		(property "P/N" "AT16-18SA"
+			(at 63.246 94.742 0)
 			(effects
 				(font
@@
 		(pin "4"
 		)
+		(pin "18"
+		)
+		(pin "15"
+		)
+		(pin "16"
+		)
+		(pin "17"
+		)
+		(pin "14"
+		)
+		(pin "13"
+		)
 		(instances

Commit message: Started on firewall
Changed lines of the file:
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@@
 		)
 		(property "P/N" "AT16-18SA"
-			(at 63.246 94.742 0)
+			(at 42.418 93.726 0)
 			(effects
 				(font
+					(size 1.27 1.27)
+				)
+			)
+		)
+		(property "Conn Name" ""
+			(at 52.07 101.6 0)
+			(effects
+				(font

Commit message: remove stag11 accu and rename comp datalogger bus
Connections:
- net CAN.FSUK.H renamed CAN.COMP.H
- net CAN.FSUK.L renamed CAN.COMP.L
- net FSUK.DL.PWR renamed COMP_DL.PWR
Changed lines of the file:
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@@
 		)
 	)
-	(label "FSUK.DL.GND"
+	(label "FSUK_DL.GND"
 		(at 53.975 99.695 0)
 		(effects
@@
 		)
 	)
-	(label "CAN.FSUK.L"
+	(label "CAN.COMP.L"
 		(at 53.9732 97.155 0)
 		(effects
@@
 		)
 	)
-	(label "CAN.FSUK.H"
+	(label "CAN.COMP.H"
 		(at 53.975 94.615 0)
 		(effects
@@
 		)
 	)
-	(label "FSUK.DL.PWR"
+	(label "COMP_DL.PWR"
 		(at 53.9732 92.075 0)
 		(effects

Commit message: Top loom and LV box?
Connections:
- net AIRBRIDGE.PWR: now reaches Conn60.13
- net CAN.T.H: now reaches Conn60.14
- net CAN.T.L: now reaches Conn60.15
- net AIRBRIDGE.GND: now reaches Conn60.16
- net R2D.GND renamed RTDS-
- net R2D.PWR renamed RTDS+
- no-connect marks 0 -> 2
Other:
- note added: "DB9"
Changed lines of the file:
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@@
 	(generator_version "9.0")
 	(paper "A4")
+	(text "DB9"
+		(exclude_from_sim no)
+		(at 222.25 131.064 0)
+		(effects
+			(font
+				(size 1.27 1.27)
+			)
+		)
+	)
 	(text "Might be\n09 9764 70 04\n\nWarwick might know?"
 		(exclude_from_sim no)
@@
 		)
 	)
+	(no_connect
+		(at 52.705 114.935)
+	)
+	(no_connect
+		(at 52.705 112.395)
+	)
 	(wire
 		(pts
@@
 	(wire
 		(pts
+			(xy 52.705 107.315) (xy 121.285 107.315)
+		)
+		(stroke
+			(width 0)
+			(type default)
+		)
+	)
+	(wire
+		(pts
 			(xy 181.61 50.8) (xy 215.9 50.8)
 		)
@@
 	(wire
 		(pts
+			(xy 124.46 130.175) (xy 201.2968 130.175)
+		)
+		(stroke
+			(width 0)
+			(type default)
+		)
+	)
+	(wire
+		(pts
 			(xy 52.705 92.075) (xy 148.59 92.075)
 		)
@@
 	(wire
 		(pts
+			(xy 201.295 132.715) (xy 121.285 132.715)
+		)
+		(stroke
+			(width 0)
+			(type default)
+		)
+	)
+	(wire
+		(pts
+			(xy 201.2968 127.635) (xy 127 127.635)
+		)
+		(stroke
+			(width 0)
+			(type default)
+		)
+	)
+	(wire
+		(pts
 			(xy 52.705 89.535) (xy 151.13 89.535)
 		)
@@
 	(wire
 		(pts
+			(xy 52.705 104.775) (xy 124.46 104.775)
+		)
+		(stroke
+			(width 0)
+			(type default)
+		)
+	)
+	(wire
+		(pts
 			(xy 151.13 95.885) (xy 214.63 95.885)
 		)
@@
 	(wire
 		(pts
+			(xy 118.11 109.855) (xy 118.11 135.255)
+		)
+		(stroke
+			(width 0)
+			(type default)
+		)
+	)
+	(wire
+		(pts
 			(xy 52.705 71.755) (xy 143.51 71.755)
 		)
@@
 	(wire
 		(pts
+			(xy 127 127.635) (xy 127 102.235)
+		)
+		(stroke
+			(width 0)
+			(type default)
+		)
+	)
+	(wire
+		(pts
 			(xy 52.705 86.995) (xy 153.67 86.995)
 		)
@@
 	(wire
 		(pts
+			(xy 124.46 104.775) (xy 124.46 130.175)
+		)
+		(stroke
+			(width 0)
+			(type default)
+		)
+	)
+	(wire
+		(pts
 			(xy 140.97 112.395) (xy 214.63 112.395)
 		)
@@
 	(wire
 		(pts
+			(xy 118.11 135.255) (xy 201.2968 135.255)
+		)
+		(stroke
+			(width 0)
+			(type default)
+		)
+	)
+	(wire
+		(pts
+			(xy 121.285 132.715) (xy 121.285 107.315)
+		)
+		(stroke
+			(width 0)
+			(type default)
+		)
+	)
+	(wire
+		(pts
 			(xy 151.13 89.535) (xy 151.13 95.885)
 		)
@@
 	(wire
 		(pts
+			(xy 52.705 102.235) (xy 127 102.235)
+		)
+		(stroke
+			(width 0)
+			(type default)
+		)
+	)
+	(wire
+		(pts
 			(xy 179.07 48.26) (xy 215.9 48.26)
+		)
+		(stroke
+			(width 0)
+			(type default)
+		)
+	)
+	(wire
+		(pts
+			(xy 52.705 109.855) (xy 118.11 109.855)
 		)
 		(stroke
@@
 		)
 	)
-	(label "R2D.PWR"
+	(label "AIRBRIDGE.PWR"
+		(at 201.2968 127.635 0)
+		(effects
+			(font
+				(size 1.27 1.27)
+			)
+			(justify left bottom)
+		)
+	)
+	(label "RTDS+"
 		(at 53.9732 86.995 0)
+		(effects
+			(font
+				(size 1.27 1.27)
+			)
+			(justify left bottom)
+		)
+	)
+	(label "CAN.T.H"
+		(at 53.975 104.775 0)
 		(effects
 			(font
@@
 		)
 	)
+	(label "AIRBRIDGE.GND"
+		(at 201.2968 135.255 0)
+		(effects
+			(font
+				(size 1.27 1.27)
+			)
+			(justify left bottom)
+		)
+	)
 	(label "SDC.FRONT"
 		(at 53.9732 74.295 0)
@@
 		)
 	)
-	(label "R2D.GND"
+	(label "RTDS-"
 		(at 53.975 89.535 0)
 		(effects
@@
 		)
 	)
+	(label "CAN.T.L"
+		(at 53.9732 107.315 0)
+		(effects
+			(font
+				(size 1.27 1.27)
+			)
+			(justify left bottom)
+		)
+	)
+	(label "CAN.T.L"
+		(at 201.295 132.715 0)
+		(effects
+			(font
+				(size 1.27 1.27)
+			)
+			(justify left bottom)
+		)
+	)
 	(label "TSAL.GND"
 		(at 200.025 84.455 0)
@@
 		)
 	)
+	(label "CAN.T.H"
+		(at 201.2968 130.175 0)
+		(effects
+			(font
+				(size 1.27 1.27)
+			)
+			(justify left bottom)
+		)
+	)
 	(label "CAN.FSUK.L"
 		(at 200.0232 109.855 0)
@@
 		)
 	)
-	(label "R2D.PWR"
+	(label "RTDS+"
 		(at 200.0232 93.345 0)
 		(effects
@@
 		)
 	)
+	(label "AIRBRIDGE.PWR"
+		(at 53.975 102.235 0)
+		(effects
+			(font
+				(size 1.27 1.27)
+			)
+			(justify left bottom)
+		)
+	)
+	(label "AIRBRIDGE.GND"
+		(at 53.975 109.855 0)
+		(effects
+			(font
+				(size 1.27 1.27)
+			)
+			(justify left bottom)
+		)
+	)
 	(label "TSAL.GRN.EN"
 		(at 54.0319 81.915 0)
@@
 		)
 	)
-	(label "R2D.GND"
+	(label "RTDS-"
 		(at 200.025 95.885 0)
 		(effects

Commit message: bunch of changes, notably rear loom
Connections:
- net CAN.T.H renamed CAN.AB.H
- net CAN.T.L renamed CAN.AB.L
Changed lines of the file:
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@@
-		)
-	)
-	(label "CAN.T.H"
-		(at 53.975 104.775 0)
-		(effects
-			(font
-				(size 1.27 1.27)
-			)
-			(justify left bottom)
 		)
 	)
@@
 	)
 	(label "CAN.T.L"
-		(at 53.9732 107.315 0)
-		(effects
-			(font
-				(size 1.27 1.27)
-			)
-			(justify left bottom)
-		)
-	)
-	(label "CAN.T.L"
 		(at 201.295 132.715 0)
 		(effects
@@
 		)
 	)
+	(label "CAN.AB.H"
+		(at 53.975 104.775 0)
+		(effects
+			(font
+				(size 1.27 1.27)
+			)
+			(justify left bottom)
+		)
+	)
 	(label "SDC.R-SW"
 		(at 200.025 50.8 0)
@@
 		(effects
 			(font
+				(size 1.27 1.27)
+			)
+			(justify left bottom)
+		)
+	)
+	(label "CAN.AB.L"
+		(at 53.975 107.315 0)
+		(effects
+			(font

Commit message: TSAL pinout
Parts:
- added J187: Conn_01x04_Socket, symbol Connector:Conn_01x04_Socket
Connections:
- net TSAL.GND: now also J187.2 (Pin_2)
- net TSAL.GRN.EN: now also J187.4 (Pin_4)
- net TSAL.PWR: now also J187.1 (Pin_1)
- net TSAL.RED.EN: now also J187.3 (Pin_3)
Other:
- moved on the sheet: Conn60
